File: Lab_01/Lab01_P06.kicad_sch (KiCad schematic)
At the start: 5 parts

Commit message: Update RC Filters
Parts:
- C61: value 6800p -> 0.0022u
- R62: value 2.4k -> 6.8k
Changed lines of the file:
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@@
       (effects (font (size 1.27 1.27)) (justify left))
     )
-    (property "Value" "6800p" (at 86.36 48.26 0)
+    (property "Value" "0.0022u" (at 86.36 48.26 0)
       (effects (font (size 1.27 1.27)) (justify left))
     )
@@
       (effects (font (size 1.27 1.27)))
     )
-    (property "Value" "2.4k" (at 68.58 30.48 90)
+    (property "Value" "6.8k" (at 68.58 30.48 90)
       (effects (font (size 1.27 1.27)))
     )

Commit message: Edit up to Question 9
Other:
- note added: "fc = 1/(2piRC) = 10.6 KHz"
- note removed: "fc = 1/(2piRC) = 9.75 KHz"
Changed lines of the file:
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@@
     (stroke (width 0) (type default))
   )
-  (text "fc = 1/(2piRC) = 9.75 KHz" (at 78.74 29.21 0)
+  (text "fc = 1/(2piRC) = 10.6 KHz" (at 78.74 29.21 0)
     (effects (font (size 1.27 1.27)) (justify left bottom))
   )
