File: Lab_01/Lab01_P07.kicad_sch (KiCad schematic)
At the start: 7 parts

Commit message: Update RC Filters
Parts:
- C71: value 6800p -> 0.0022u
- C72: value 0.068u -> 220p
- R72: value 2.4k -> 6.8k
- R73: value 2.4k -> 680k
Other:
- note added: "STAGE 1 LP 10.64 KHz"
- note added: "STAGE 2 HP 1064 Hz"
- note removed: "STAGE 1 LP 9.75 KHz"
- note removed: "STAGE 2 HP 975 Hz"
Changed lines of the file:
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@@
     (stroke (width 0) (type default))
   )
-  (text "STAGE 1\nLP\n9.75 KHz" (at 85.09 38.1 0)
+  (text "STAGE 1\nLP\n10.64 KHz" (at 85.09 38.1 0)
     (effects (font (size 1.27 1.27)) (justify right bottom))
   )
-  (text "STAGE 2\nHP\n975 Hz" (at 109.22 38.1 0)
+  (text "STAGE 2\nHP\n1064 Hz" (at 109.22 38.1 0)
     (effects (font (size 1.27 1.27)) (justify right bottom))
   )
@@
       (effects (font (size 1.27 1.27)))
     )
-    (property "Value" "2.4k" (at 69.85 38.1 90)
+    (property "Value" "6.8k" (at 69.85 38.1 90)
       (effects (font (size 1.27 1.27)))
     )
@@
       (effects (font (size 1.27 1.27)))
     )
-    (property "Value" "0.068u" (at 95.25 36.83 90)
+    (property "Value" "220p" (at 95.25 36.83 90)
       (effects (font (size 1.27 1.27)))
     )
@@
   )
   (symbol (lib_id "Device:C") (at 76.2 52.07 0) (unit 1)
-    (in_bom yes) (on_board yes) (dnp no) (fields_autoplaced)
-    (property "Reference" "C71" (at 80.01 50.8 0)
-      (effects (font (size 1.27 1.27)) (justify left))
-    )
-    (property "Value" "6800p" (at 80.01 53.34 0)
+    (in_bom yes) (on_board yes) (dnp no)
+    (property "Reference" "C71" (at 80.01 52.07 0)
+      (effects (font (size 1.27 1.27)) (justify left))
+    )
+    (property "Value" "0.0022u" (at 77.47 54.61 0)
       (effects (font (size 1.27 1.27)) (justify left))
     )
@@
   )
   (symbol (lib_id "Device:R") (at 102.87 52.07 180) (unit 1)
-    (in_bom yes) (on_board yes) (dnp no) (fields_autoplaced)
+    (in_bom yes) (on_board yes) (dnp no)
     (property "Reference" "R73" (at 105.41 50.8 0)
       (effects (font (size 1.27 1.27)) (justify right))
     )
-    (property "Value" "2.4k" (at 105.41 53.34 0)
-      (effects (font (size 1.27 1.27)) (justify right))
-    )
+    (property "Value" "680k" (at 105.41 53.34 0)
+      (effects (font (size 1.27 1.27)) (justify right))
+    )

Commit message: Edit up to Question 9
Parts:
- removed C71: 0.0022u, symbol Device:C
- removed R72: 6.8k, symbol Device:R
- added C1: 220p, symbol Device:C
- added R1: 680k, symbol Device:R
- C72: value 220p -> 0.0022u
- R73: value 680k -> 6.8k
Connections:
- net GND: now also C1.2
- net Vout: now also C1.1, R1.2; no longer C72.2, R73.2
- net Vsin7: now also C72.1
- new net: C72.2, R1.1, R73.2
Other:
- moved on the sheet: C72, R73
