File: Lab_02/Lab02.kicad_sch (KiCad schematic)
At the start: 0 parts

Commit message: Finish Lab 02 Saturday Schematics
Parts:
- added V1, V2: 15, symbol Simulation_SPICE:VDC
Connections:
- new net +15V: V1.1
- new net -15V: V2.1
- new net GND: V1.2, V2.2
Other:
- company: (none) -> Jim Horwitz & Mark Vaughn, Jork Incorporated
Changed lines of the file:
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@@
 (kicad_sch (version 20230121) (generator eeschema)
   (paper "A4")
+  (title_block
+    (rev "0")
+    (company "Jim Horwitz & Mark Vaughn, Jork Incorporated")
+  )
+  (junction (at 38.1 158.75) (diameter 0) (color 0 0 0 0)
+  )
+  (wire (pts (xy 38.1 170.18) (xy 38.1 171.45))
+    (stroke (width 0) (type default))
+  )
+  (wire (pts (xy 29.21 160.02) (xy 29.21 158.75))
+    (stroke (width 0) (type default))
+  )
+  (wire (pts (xy 38.1 158.75) (xy 38.1 157.48))
+    (stroke (width 0) (type default))
+  )
+  (wire (pts (xy 38.1 146.05) (xy 38.1 147.32))
+    (stroke (width 0) (type default))
+  )
+  (wire (pts (xy 29.21 158.75) (xy 38.1 158.75))
+    (stroke (width 0) (type default))
+  )
+  (wire (pts (xy 38.1 158.75) (xy 38.1 160.02))
+    (stroke (width 0) (type default))
+  )
+  (symbol (lib_id "Simulation_SPICE:VDC") (at 38.1 165.1 0) (mirror x) (unit 1)
+    (in_bom yes) (on_board yes) (dnp no)
+    (property "Reference" "V2" (at 41.91 166.4058 0)
+      (effects (font (size 1.27 1.27)) (justify left))
+    )
+    (property "Value" "15" (at 41.91 163.8658 0)
+      (effects (font (size 1.27 1.27)) (justify left))
+    )
+    (property "Footprint" "" (at 38.1 165.1 0)
+      (effects (font (size 1.27 1.27)) hide)
+    )
+    (property "Datasheet" "~" (at 38.1 165.1 0)
+      (effects (font (size 1.27 1.27)) hide)
+    )
+    (property "Sim.Pins" "1=+ 2=-" (at 38.1 165.1 0)
+      (effects (font (size 1.27 1.27)) hide)
+    )
+    (property "Sim.Type" "DC" (at 38.1 165.1 0)
+      (effects (font (size 1.27 1.27)) hide)
+    )
+    (property "Sim.Device" "V" (at 38.1 165.1 0)
+      (effects (font (size 1.27 1.27)) (justify left) hide)
+    )
+    (pin "1")
+    (pin "2")
+    (instances
+      (project "Lab02"
+        (path "/b848c9df-85a0-48ab-ac89-72f46cf8e040"
+          (reference "V2") (unit 1)
+        )
+      )
+    )
+  )
+  (symbol (lib_id "power:GND") (at 29.21 160.02 0) (unit 1)
+    (in_bom yes) (on_board yes) (dnp no)
+    (property "Reference" "#PWR012" (at 29.21 166.37 0)
+      (effects (font (size 1.27 1.27)) hide)
+    )
+    (property "Value" "GND" (at 29.21 163.83 0)
+      (effects (font (size 1.27 1.27)))
+    )
+    (property "Footprint" "" (at 29.21 160.02 0)
+      (effects (font (size 1.27 1.27)) hide)
+    )
+    (property "Datasheet" "" (at 29.21 160.02 0)
+      (effects (font (size 1.27 1.27)) hide)
+    )
+    (pin "1")
+    (instances
+      (project "Lab02"
+        (path "/b848c9df-85a0-48ab-ac89-72f46cf8e040"
+          (reference "#PWR012") (unit 1)
+        )
+      )
+    )
+  )
+  (symbol (lib_id "Simulation_SPICE:VDC") (at 38.1 152.4 0) (unit 1)
+    (in_bom yes) (on_board yes) (dnp no) (fields_autoplaced)
+    (property "Reference" "V1" (at 41.91 151.0942 0)
+      (effects (font (size 1.27 1.27)) (justify left))
+    )
+    (property "Value" "15" (at 41.91 153.6342 0)
+      (effects (font (size 1.27 1.27)) (justify left))
+    )
+    (property "Footprint" "" (at 38.1 152.4 0)
+      (effects (font (size 1.27 1.27)) hide)
+    )
+    (property "Datasheet" "~" (at 38.1 152.4 0)
+      (effects (font (size 1.27 1.27)) hide)
+    )
+    (property "Sim.Pins" "1=+ 2=-" (at 38.1 152.4 0)
+      (effects (font (size 1.27 1.27)) hide)
+    )
+    (property "Sim.Type" "DC" (at 38.1 152.4 0)
+      (effects (font (size 1.27 1.27)) hide)
+    )
+    (property "Sim.Device" "V" (at 38.1 152.4 0)
+      (effects (font (size 1.27 1.27)) (justify left) hide)
+    )
+    (pin "1")
+    (pin "2")
+    (instances
+      (project "Lab02"
+        (path "/b848c9df-85a0-48ab-ac89-72f46cf8e040"
+          (reference "V1") (unit 1)
+        )
+      )
+    )
+  )
+  (symbol (lib_id "power:+15V") (at 38.1 146.05 0) (unit 1)
+    (in_bom yes) (on_board yes) (dnp no)
+    (property "Reference" "#PWR017" (at 38.1 149.86 0)
+      (effects (font (size 1.27 1.27)) hide)
+    )
+    (property "Value" "+15V" (at 38.1 142.24 0)
+      (effects (font (size 1.27 1.27)))
+    )
+    (property "Footprint" "" (at 38.1 146.05 0)
+      (effects (font (size 1.27 1.27)) hide)
+    )
+    (property "Datasheet" "" (at 38.1 146.05 0)
+      (effects (font (size 1.27 1.27)) hide)
+    )
+    (pin "1")
+    (instances
+      (project "Lab02"
+        (path "/b848c9df-85a0-48ab-ac89-72f46cf8e040"
+          (reference "#PWR017") (unit 1)
+        )
+      )
+    )
+  )
+  (symbol (lib_id "power:-15V") (at 38.1 171.45 0) (mirror x) (unit 1)
+    (in_bom yes) (on_board yes) (dnp no)
+    (property "Reference" "#PWR015" (at 38.1 173.99 0)
+      (effects (font (size 1.27 1.27)) hide)
+    )
+    (property "Value" "-15V" (at 38.1 175.26 0)
+      (effects (font (size 1.27 1.27)))
+    )
+    (property "Footprint" "" (at 38.1 171.45 0)
+      (effects (font (size 1.27 1.27)) hide)
+    )
+    (property "Datasheet" "" (at 38.1 171.45 0)
+      (effects (font (size 1.27 1.27)) hide)
+    )
+    (pin "1")
+    (instances
+      (project "Lab02"
+        (path "/b848c9df-85a0-48ab-ac89-72f46cf8e040"
+          (reference "#PWR015") (unit 1)
+        )
+      )
+    )
+  )
   (sheet (at 87.63 55.88) (size 55.88 39.37) (fields_autoplaced)
     (stroke (width 0.1524) (type solid))
