File: Lab_02/Lab02.kicad_sch (KiCad schematic)
At the start: 0 parts

Commit message: q4 ss done
Changed lines of the file:
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@@
     )
   )
-  (sheet (at 40.64 35.56) (size 55.88 39.37) (fields_autoplaced)
+  (sheet (at 87.63 55.88) (size 55.88 39.37) (fields_autoplaced)
     (stroke (width 0.1524) (type solid))
     (fill (color 0 0 0 0.0000))
-    (property "Sheetname" "SS_Q4" (at 40.64 34.8484 0)
+    (property "Sheetname" "SS_Q4" (at 87.63 55.1684 0)
       (effects (font (size 1.27 1.27)) (justify left bottom))
     )
-    (property "Sheetfile" "SS_Q4.kicad_sch" (at 40.64 75.5146 0)
+    (property "Sheetfile" "SS_Q4.kicad_sch" (at 87.63 95.8346 0)
       (effects (font (size 1.27 1.27)) (justify left top))
     )

Commit message: Organize Saturday Schematic Sheets
Other:
- added sheet Problem 3 (Lab02_P03.kicad_sch)
Changed lines of the file:
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@@
 (kicad_sch (version 20230121) (generator eeschema)
   (paper "A4")
-  (sheet (at 370.84 167.64) (size 12.7 3.81) (fields_autoplaced)
-    (stroke (width 0.1524) (type solid))
-    (fill (color 0 0 0 0.0000))
-    (property "Sheetname" "SS_Q4" (at 370.84 166.9284 0)
-      (effects (font (size 1.27 1.27)) (justify left bottom))
-    )
-    (property "Sheetfile" "SS_Q4.kicad_sch" (at 370.84 172.0346 0)
-      (effects (font (size 1.27 1.27)) (justify left top))
-    )
-    (instances
-      (project "Lab02"
-        (path "/b848c9df-85a0-48ab-ac89-72f46cf8e040" (page "2"))
-      )
-    )
-  )
   (sheet (at 87.63 55.88) (size 55.88 39.37) (fields_autoplaced)
     (stroke (width 0.1524) (type solid))
@@
       (effects (font (size 1.27 1.27)) (justify left top))
     )
+    (instances
+      (project "Lab02"
+        (path "/b848c9df-85a0-48ab-ac89-72f46cf8e040" (page "4"))
+      )
+    )
+  )
+  (sheet (at 170.18 55.88) (size 59.69 38.1) (fields_autoplaced)
+    (stroke (width 0.1524) (type solid))
+    (fill (color 0 0 0 0.0000))
+    (property "Sheetname" "Problem 3" (at 170.18 55.1684 0)
+      (effects (font (size 1.27 1.27)) (justify left bottom))
+    )
+    (property "Sheetfile" "Lab02_P03.kicad_sch" (at 170.18 94.5646 0)
+      (effects (font (size 1.27 1.27)) (justify left top))
+    )

Commit message: writeup
Other:
- added sheet Problem 1 (Problem_1.kicad_sch)
- added sheet Problem 2 (Problem_2.kicad_sch)
Changed lines of the file:
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@@
     )
   )
-  (sheet (at 170.18 55.88) (size 59.69 38.1) (fields_autoplaced)
+  (sheet (at 170.18 55.88) (size 55.88 38.1) (fields_autoplaced)
     (stroke (width 0.1524) (type solid))
     (fill (color 0 0 0 0.0000))
@@
       )
     )
+  )
+  (sheet (at 170.18 100.33) (size 55.88 33.02) (fields_autoplaced)
+    (stroke (width 0.1524) (type solid))
+    (fill (color 0 0 0 0.0000))
+    (property "Sheetname" "Problem 1" (at 170.18 99.6184 0)
+      (effects (font (size 1.27 1.27)) (justify left bottom))
+    )
+    (property "Sheetfile" "Problem_1.kicad_sch" (at 170.18 133.9346 0)
+      (effects (font (size 1.27 1.27)) (justify left top))
+    )
+    (instances
+      (project "Lab02"
+        (path "/b848c9df-85a0-48ab-ac89-72f46cf8e040" (page "2"))
+      )
+    )
+  )
+  (sheet (at 87.63 100.33) (size 55.88 33.02) (fields_autoplaced)
+    (stroke (width 0.1524) (type solid))
+    (fill (color 0 0 0 0.0000))
+    (property "Sheetname" "Problem 2" (at 87.63 99.6184 0)
+      (effects (font (size 1.27 1.27)) (justify left bottom))
+    )
+    (property "Sheetfile" "Problem_2.kicad_sch" (at 87.63 133.9346 0)
+      (effects (font (size 1.27 1.27)) (justify left top))
+    )
+    (instances
+      (project "Lab02"
+        (path "/b848c9df-85a0-48ab-ac89-72f46cf8e040" (page "4"))
+      )
+    )
