File: Lab_02/Lab02_P03.kicad_sch (KiCad schematic)
At the start: 0 parts

Commit message: Finish Lab 02 Saturday Schematics
Parts:
- added R301, R306, R307: R, symbol Device:R
- added R302: R/2, symbol Device:R
- added R303, R304, R305: 2R, symbol Device:R
- added SW301: SW_SPST, symbol Switch:SW_SPST
- added U301, U302: LM741, symbol Amplifier_Operational:LM741
- added V301: 1, symbol Simulation_SPICE:VDC
- added V302: 2, symbol Simulation_SPICE:VDC
- added V303: 5, symbol Simulation_SPICE:VDC
Connections:
- new net: R305.2, SW301.1 (A)
- new net: R304.2, R306.1, SW301.2 (B), U301.6
- new net: R301.2, R302.2, R303.2, R304.1, R305.1, U301.2 (-)
- new net: R306.2, R307.1, U302.2 (-)
- new net +15V: U301.7 (V+), U302.7 (V+)
- new net -15V: U301.4 (V-), U302.4 (V-)
- new net GND: U301.3 (+), U302.3 (+), V301.2, V302.2, V303.2
- new net VA: R301.1, V301.1
- new net VB: R302.1, V302.1
- new net VC: R303.1, V303.1
- new net Vout: R307.2, U302.6
Other:
- note added: "Closed-loop gain is halved when switch SW301 is closed"
- note added: "INVERTING AMP UNITY GAIN"
- note added: "SUMMING AMP Gc = 2V/V"
- company: (none) -> Jim Horwitz & Mark Vaughn, Jork Incorporated
- title: (none) -> Weighted Voltage Summer

Commit message: Finish Lab 02
Parts:
- R301: value R -> 5.1K
- R302: value R/2 -> 2.4K
- R303, R304, R305: value 2R -> 10K
- R306, R307: value R -> 6.8K
Changed lines of the file:
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@@
   (title_block
     (title "Weighted Voltage Summer")
-    (date "2024-01-27")
-    (rev "0")
+    (date "2024-01-31")
+    (rev "1")
     (company "Jim Horwitz & Mark Vaughn, Jork Incorporated")
+    (comment 1 "All resistors 5% tolerance")
   )
   (junction (at 62.23 39.37) (diameter 0) (color 0 0 0 0)
@@
       (effects (font (size 1.27 1.27)))
     )
-    (property "Value" "2R" (at 49.53 59.69 90)
+    (property "Value" "10K" (at 49.53 59.69 90)
       (effects (font (size 1.27 1.27)))
     )
@@
       (effects (font (size 1.27 1.27)))
     )
-    (property "Value" "R" (at 116.84 41.91 90)
+    (property "Value" "6.8K" (at 116.84 41.91 90)
       (effects (font (size 1.27 1.27)))
     )
@@
       (effects (font (size 1.27 1.27)))
     )
-    (property "Value" "R" (at 97.79 55.88 90)
+    (property "Value" "6.8K" (at 97.79 55.88 90)
       (effects (font (size 1.27 1.27)))
     )
@@
       (effects (font (size 1.27 1.27)))
     )
-    (property "Value" "R" (at 49.53 46.99 90)
+    (property "Value" "5.1K" (at 49.53 46.99 90)
       (effects (font (size 1.27 1.27)))
     )
@@
       (effects (font (size 1.27 1.27)))
     )
-    (property "Value" "2R" (at 73.66 39.37 90)
+    (property "Value" "10K" (at 73.66 39.37 90)
       (effects (font (size 1.27 1.27)))
     )
@@
       (effects (font (size 1.27 1.27)))
     )
-    (property "Value" "2R" (at 67.31 33.02 90)
+    (property "Value" "10K" (at 67.31 33.02 90)
       (effects (font (size 1.27 1.27)))
     )
@@
       (effects (font (size 1.27 1.27)))
     )
-    (property "Value" "R/2" (at 49.53 53.34 90)
-      (effects (font (size 1.27 1.27)))
-    )
+    (property "Value" "2.4K" (at 49.53 53.34 90)
+      (effects (font (size 1.27 1.27)))
+    )
