File: Lab_02/Problem_1.kicad_sch (KiCad schematic)
At the start: 3 parts, among them U1 LM741

Commit message: Finish Lab 02
Other:
- company: (none) -> Jim Horwitz & Mark Vaughn, Jork Incorporated
Changed lines of the file:
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@@
 (kicad_sch (version 20230121) (generator eeschema)
   (paper "A4")
+  (title_block
+    (company "Jim Horwitz & Mark Vaughn, Jork Incorporated")
+  )
   (junction (at 52.07 57.15) (diameter 0) (color 0 0 0 0)
   )
@@
       (effects (font (size 1.27 1.27)) hide)
     )
-    (pin "7")
     (pin "1")
+    (pin "2")
+    (pin "3")
+    (pin "4")
     (pin "5")
     (pin "6")
+    (pin "7")
     (pin "8")
-    (pin "2")
-    (pin "4")
-    (pin "3")
     (instances
       (project "Lab02"
