File: Lab_02/Problem_2.kicad_sch (KiCad schematic)
At the start: 0 parts

Commit message: Finish Lab 02
Parts:
- added C201, C202: 0.22uF, symbol Device:C
- added R201: 1K, symbol Device:R
- added R202, R207, R5: 1M, symbol Device:R
- added R203, R204: 100, symbol Device:R
- added R205, R206: 15K, symbol Device:R
- added R208: 100K, symbol Device:R
- added U301 (x5): LM741, symbol Amplifier_Operational:LM741
Connections:
- new net: R204.2, R206.1, R208.1
- new net: C202.1, R5.2, U301.2 (-)
- new net: R207.1, U301.6
- new net: C201.1, R207.2, U301.2 (-)
- new net: R201.2, R202.1, U301.2 (-)
- new net: R203.2, R205.1
- new net: R206.2, U301.3 (+)
- new net: R205.2, U301.2 (-)
- new net +15V: U301.7 (V+), U301.7 (V+), U301.7 (V+), U301.7 (V+), U301.7 (V+)
- new net -15V: U301.4 (V-), U301.4 (V-), U301.4 (V-), U301.4 (V-), U301.4 (V-)
- new net -VOUT: R202.2, U301.6
- new net GND: R201.1, R203.1, R204.1, U301.3 (+), U301.3 (+), U301.3 (+)
- new net VIN: R5.1, U301.3 (+)
- new net VOUT: U301.2 (-), U301.6
- new net Vout: C201.2, C202.2, R208.2, U301.6, U301.6
- no-connect marks 0 -> 1
Other:
- note added: "-10V"
- note added: "1/RC = 5Hz"
- note added: "10V"
- note added: "= 1000 * Voffset"
- note added: "= VIN + Voffset"
- note added: ">25ms"
- note added: "DEVICE UNDER TEST"
- note added: "Ibias = C202 * -dVout/dt"
- note added: "PART 1"
- note added: "PARTS 2-4"
- note added: "Remove generator"
- note added: "Short across R205 or R206 to measure bias current through opposite input"
- note added: "Vout ranges from 0 to -12V Ibias = -Vout/15M"
- company: (none) -> Jim Horwitz & Mark Vaughn, Jork Incorporated
