File: Lab_02/SS_Q4.kicad_sch (KiCad schematic)
At the start: 16 parts

Commit message: q4 ss done
Parts:
- added C10, C12, C14, C16: C, symbol Device:C
- added R18, R20, R22, R24, R27, R28, R30, R32: R, symbol Device:R
- added U? (x3): LM741, symbol Amplifier_Operational:LM741
Connections:
- net GND: now also C12.1, C16.1, R32.2, U?.3 (+), U?.3 (+), U?.3 (+)
- net VCC: now also U?.7 (V+), U?.7 (V+), U?.7 (V+)
- net VEE: now also U?.4 (V-), U?.4 (V-), U?.4 (V-)
- net Vi: now also R18.1, R27.1
- net Vo: now also R16.1, U?.6, R22.2, R30.2, U?.6, U?.6
- new net: C10.1, R20.1, U?.6
- new net: C10.2, R18.2, U?.2 (-)
- new net: C12.2, R20.2, R24.1
- new net: R22.1, R24.2, U?.2 (-)
- new net: C14.1, R27.2, U?.2 (-)
- new net: C14.2, C16.2, R28.1
- new net: R28.2, R30.1, R32.1
- no-connect marks 8 -> 14

Commit message: Finish Lab 02 Saturday Schematics
Other:
- company: (none) -> Jim Horwitz & Mark Vaughn, Jork Incorporated
- title: (none) -> Active Bandpass Filter Topologies
- moved on the sheet: C10, C12, C14, C16, C2, C4, C6, C8, R10, R12, R14, R16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

Commit message: lab 3 init
Parts:
- removed C10, C12, C14, C16, C2, C4, C6, C8: C, symbol Device:C
- removed R10, R12, R14, R16, R18, R20, R22, R24, R27, R28, R30, R32, R4, R6, R8: R, symbol Device:R
- removed U? (x6): LM741, symbol Amplifier_Operational:LM741
Connections:
- net Vo: now also R2.1
- net at U?.2 (-): now also R2.2
- no-connect marks 14 -> 2
Other:
- note removed: "Gain"
- note removed: "HPF"
- note removed: "LPF"
