File: Lab_03/KiCad/q1.kicad_sch (KiCad schematic)
At the start: 8 parts, among them U1 LM339, U2 LM339

Commit message: 1 done
Parts:
- added R5: 1M, symbol Device:R
- added R6: 100K, symbol Device:R
Connections:
- net vin: now also R6.2; no longer U2.5 (+)
- net vout: now also R5.1
- new net: R5.2, R6.1, U2.5 (+)
Other:
- note added: "1B"
- moved on the sheet: R3, R4, RV2, U2A
