File: Lab_03/KiCad/q1.kicad_sch (KiCad schematic)
At the start: 10 parts, among them U1 LM339, U2 LM339

Commit message: Update earlier parts of lab03
Parts:
- renumbered R1 to R301, R2 to R302, R3 to R303, R6 to R304, R5 to R305, R4 to R306, RV1 to RV301, RV2 to RV302, U1 to U301, U2 to U302
Changed lines of the file:
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@@
   (symbol (lib_id "power:+10V") (at 55.88 66.04 0) (unit 1)
     (in_bom yes) (on_board yes) (dnp no) (fields_autoplaced)
-    (property "Reference" "#PWR01" (at 55.88 69.85 0)
+    (property "Reference" "#PWR0301" (at 55.88 69.85 0)
       (effects (font (size 1.27 1.27)) hide)
     )
@@
       (project "Lab03"
         (path "/0f3a9aa4-582a-427a-a342-2cdf273d26d7/efced3a7-3a3b-4a68-adb6-f42376b52d74"
-          (reference "#PWR01") (unit 1)
+          (reference "#PWR0301") (unit 1)
         )
       )
@@
   (symbol (lib_id "Device:R") (at 86.36 73.66 0) (unit 1)
     (in_bom yes) (on_board yes) (dnp no)
-    (property "Reference" "R2" (at 88.9 72.39 0)
+    (property "Reference" "R302" (at 88.9 72.39 0)
       (effects (font (size 1.27 1.27)) (justify left))
     )
@@
       (project "Lab03"
         (path "/0f3a9aa4-582a-427a-a342-2cdf273d26d7/efced3a7-3a3b-4a68-adb6-f42376b52d74"
-          (reference "R2") (unit 1)
+          (reference "R302") (unit 1)
         )
       )
@@
   (symbol (lib_id "Device:R") (at 153.67 76.2 270) (mirror x) (unit 1)
     (in_bom yes) (on_board yes) (dnp no)
-    (property "Reference" "R6" (at 154.94 73.66 0)
+    (property "Reference" "R304" (at 154.94 73.66 0)
       (effects (font (size 1.27 1.27)) (justify left))
     )
@@
       (project "Lab03"
         (path "/0f3a9aa4-582a-427a-a342-2cdf273d26d7/efced3a7-3a3b-4a68-adb6-f42376b52d74"
-          (reference "R6") (unit 1)
+          (reference "R304") (unit 1)
         )
       )
@@
   (symbol (lib_id "Comparator:LM339") (at 76.2 78.74 0) (unit 1)
     (in_bom yes) (on_board yes) (dnp no) (fields_autoplaced)
-    (property "Reference" "U1" (at 76.2 68.58 0)
+    (property "Reference" "U301" (at 76.2 68.58 0)
       (effects (font (size 1.27 1.27)))
     )
@@
       (project "Lab03"
         (path "/0f3a9aa4-582a-427a-a342-2cdf273d26d7/efced3a7-3a3b-4a68-adb6-f42376b52d74"
-          (reference "U1") (unit 1)
+          (reference "U301") (unit 1)
         )
       )
@@
   (symbol (lib_id "Comparator:LM339") (at 168.91 78.74 0) (unit 1)
     (in_bom yes) (on_board yes) (dnp no) (fields_autoplaced)
-    (property "Reference" "U2" (at 168.91 68.58 0)
+    (property "Reference" "U302" (at 168.91 68.58 0)
       (effects (font (size 1.27 1.27)))
     )
@@
       (project "Lab03"
         (path "/0f3a9aa4-582a-427a-a342-2cdf273d26d7/efced3a7-3a3b-4a68-adb6-f42376b52d74"
-          (reference "U2") (unit 1)
+          (reference "U302") (unit 1)
         )
       )
@@
   (symbol (lib_id "Device:R") (at 55.88 71.12 0) (mirror y) (unit 1)
     (in_bom yes) (on_board yes) (dnp no)
-    (property "Reference" "R1" (at 53.34 69.85 0)
+    (property "Reference" "R301" (at 53.34 69.85 0)
       (effects (font (size 1.27 1.27)) (justify left))
     )
@@
       (project "Lab03"
         (path "/0f3a9aa4-582a-427a-a342-2cdf273d26d7/efced3a7-3a3b-4a68-adb6-f42376b52d74"
-          (reference "R1") (unit 1)
+          (reference "R301") (unit 1)
         )
       )
@@
   (symbol (lib_id "Device:R") (at 135.89 71.12 0) (mirror y) (unit 1)
     (in_bom yes) (on_board yes) (dnp no)
-    (property "Reference" "R3" (at 133.35 69.85 0)
+    (property "Reference" "R303" (at 133.35 69.85 0)
       (effects (font (size 1.27 1.27)) (justify left))
     )
@@
       (project "Lab03"
         (path "/0f3a9aa4-582a-427a-a342-2cdf273d26d7/efced3a7-3a3b-4a68-adb6-f42376b52d74"
-          (reference "R3") (unit 1)
+          (reference "R303") (unit 1)
         )
       )
@@
   (symbol (lib_id "Device:R_Potentiometer") (at 55.88 81.28 0) (mirror x) (unit 1)
     (in_bom yes) (on_board yes) (dnp no)
-    (property "Reference" "RV1" (at 53.34 80.01 0)
+    (property "Reference" "RV301" (at 53.34 80.01 0)
       (effects (font (size 1.27 1.27)) (justify right))
     )
@@
       (project "Lab03"
         (path "/0f3a9aa4-582a-427a-a342-2cdf273d26d7/efced3a7-3a3b-4a68-adb6-f42376b52d74"
-          (reference "RV1") (unit 1)
+          (reference "RV301") (unit 1)
         )
       )
@@
   (symbol (lib_id "power:GND") (at 135.89 86.36 0) (unit 1)
     (in_bom yes) (on_board yes) (dnp no) (fields_autoplaced)
-    (property "Reference" "#PWR06" (at 135.89 92.71 0)
+    (property "Reference" "#PWR0305" (at 135.89 92.71 0)
       (effects (font (size 1.27 1.27)) hide)
     )
@@
       (project "Lab03"
         (path "/0f3a9aa4-582a-427a-a342-2cdf273d26d7/efced3a7-3a3b-4a68-adb6-f42376b52d74"
-          (reference "#PWR06") (unit 1)
+          (reference "#PWR0305") (unit 1)
         )
       )
@@
   (symbol (lib_id "power:+10V") (at 86.36 68.58 0) (unit 1)
     (in_bom yes) (on_board yes) (dnp no) (fields_autoplaced)
-    (property "Reference" "#PWR03" (at 86.36 72.39 0)
+    (property "Reference" "#PWR0303" (at 86.36 72.39 0)
       (effects (font (size 1.27 1.27)) hide)
     )
@@
       (project "Lab03"
         (path "/0f3a9aa4-582a-427a-a342-2cdf273d26d7/efced3a7-3a3b-4a68-adb6-f42376b52d74"
-          (reference "#PWR03") (unit 1)
+          (reference "#PWR0303") (unit 1)
         )
       )
@@
   (symbol (lib_id "power:+10V") (at 182.88 68.58 0) (unit 1)
     (in_bom yes) (on_board yes) (dnp no) (fields_autoplaced)
-    (property "Reference" "#PWR05" (at 182.88 72.39 0)
+    (property "Reference" "#PWR0306" (at 182.88 72.39 0)
       (effects (font (size 1.27 1.27)) hide)
     )
@@
       (project "Lab03"
         (path "/0f3a9aa4-582a-427a-a342-2cdf273d26d7/efced3a7-3a3b-4a68-adb6-f42376b52d74"
-          (reference "#PWR05") (unit 1)
+          (reference "#PWR0306") (unit 1)
         )
       )
@@
   (symbol (lib_id "Device:R") (at 168.91 64.77 270) (mirror x) (unit 1)
     (in_bom yes) (on_board yes) (dnp no)
-    (property "Reference" "R5" (at 170.18 62.23 0)
+    (property "Reference" "R305" (at 170.18 62.23 0)
       (effects (font (size 1.27 1.27)) (justify left))
     )
@@
       (project "Lab03"
         (path "/0f3a9aa4-582a-427a-a342-2cdf273d26d7/efced3a7-3a3b-4a68-adb6-f42376b52d74"
-          (reference "R5") (unit 1)
+          (reference "R305") (unit 1)
         )
       )
@@
   (symbol (lib_id "power:GND") (at 55.88 86.36 0) (unit 1)
     (in_bom yes) (on_board yes) (dnp no) (fields_autoplaced)
-    (property "Reference" "#PWR02" (at 55.88 92.71 0)
+    (property "Reference" "#PWR0302" (at 55.88 92.71 0)
       (effects (font (size 1.27 1.27)) hide)
     )
@@
       (project "Lab03"
         (path "/0f3a9aa4-582a-427a-a342-2cdf273d26d7/efced3a7-3a3b-4a68-adb6-f42376b52d74"
-          (reference "#PWR02") (unit 1)
+          (reference "#PWR0302") (unit 1)
         )
       )
@@
   (symbol (lib_id "Device:R") (at 182.88 73.66 0) (unit 1)
     (in_bom yes) (on_board yes) (dnp no)
-    (property "Reference" "R4" (at 185.42 72.39 0)
+    (property "Reference" "R306" (at 185.42 72.39 0)
       (effects (font (size 1.27 1.27)) (justify left))
     )
@@
       (project "Lab03"
         (path "/0f3a9aa4-582a-427a-a342-2cdf273d26d7/efced3a7-3a3b-4a68-adb6-f42376b52d74"
-          (reference "R4") (unit 1)
+          (reference "R306") (unit 1)
         )
       )
@@
   (symbol (lib_id "Device:R_Potentiometer") (at 135.89 81.28 0) (mirror x) (unit 1)
     (in_bom yes) (on_board yes) (dnp no)
-    (property "Reference" "RV2" (at 133.35 80.01 0)
+    (property "Reference" "RV302" (at 133.35 80.01 0)
       (effects (font (size 1.27 1.27)) (justify right))
     )
@@
       (project "Lab03"
         (path "/0f3a9aa4-582a-427a-a342-2cdf273d26d7/efced3a7-3a3b-4a68-adb6-f42376b52d74"
-          (reference "RV2") (unit 1)
+          (reference "RV302") (unit 1)
         )
       )
@@
   (symbol (lib_id "power:+10V") (at 135.89 66.04 0) (unit 1)
     (in_bom yes) (on_board yes) (dnp no) (fields_autoplaced)
-    (property "Reference" "#PWR04" (at 135.89 69.85 0)
+    (property "Reference" "#PWR0304" (at 135.89 69.85 0)
       (effects (font (size 1.27 1.27)) hide)
     )
@@
       (project "Lab03"
         (path "/0f3a9aa4-582a-427a-a342-2cdf273d26d7/efced3a7-3a3b-4a68-adb6-f42376b52d74"
-          (reference "#PWR04") (unit 1)
-        )
-      )
+          (reference "#PWR0304") (unit 1)
+        )
+      )
