File: Lab_03/KiCad/part3.kicad_sch (KiCad schematic)
At the start: 19 parts, among them U3 LM741, U5 LM339, U7 LM339

Commit message: tweaks
Parts:
- removed U3 (x2): LM741, symbol Amplifier_Operational:LM741
- added U4, U6: LM324, symbol Amplifier_Operational:LM324
Connections:
- net GND: now also U6.2 (-)
- net vin: now also U4.3 (+)
- net at C1.2, R14.2: now also U6.3 (+)
- net at D3.2 (A), R14.1: now also U6.1
- net at C1.1, D1.1 (K), R10.1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: now also U4.2 (-)
- net at D1.2 (A): now also U4.1
- no-connect marks 4 -> 0

Commit message: tweaks
Connections:
- net at D3.2 (A), U6.1: no longer R14.1
- net at C1.2, D3.1 (K), R15.2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: now also R14.1
Changed lines of the file:
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@@
   (junction (at 73.66 74.93) (diameter 0) (color 0 0 0 0)
-  )
-  (junction (at 193.04 80.01) (diameter 0) (color 0 0 0 0)
   )
   (junction (at 83.82 74.93) (diameter 0) (color 0 0 0 0)
@@
   )
   (junction (at 69.85 74.93) (diameter 0) (color 0 0 0 0)
+  )
+  (junction (at 204.47 80.01) (diameter 0) (color 0 0 0 0)
   )
   (junction (at 146.05 77.47) (diameter 0) (color 0 0 0 0)
@@
     (stroke (width 0) (type default))
   )
-  (wire (pts (xy 203.2 80.01) (xy 207.01 80.01))
+  (wire (pts (xy 203.2 80.01) (xy 204.47 80.01))
     (stroke (width 0) (type default))
   )
@@
     (stroke (width 0) (type default))
   )
+  (wire (pts (xy 185.42 60.96) (xy 204.47 60.96))
+    (stroke (width 0) (type default))
+  )
   (wire (pts (xy 107.95 88.9) (xy 109.22 88.9))
     (stroke (width 0) (type default))
@@
     (stroke (width 0) (type default))
   )
-  (wire (pts (xy 190.5 80.01) (xy 193.04 80.01))
+  (wire (pts (xy 171.45 77.47) (xy 175.26 77.47))
     (stroke (width 0) (type default))
   )
-  (wire (pts (xy 171.45 77.47) (xy 175.26 77.47))
+  (wire (pts (xy 204.47 80.01) (xy 204.47 60.96))
     (stroke (width 0) (type default))
   )
@@
     (stroke (width 0) (type default))
   )
+  (wire (pts (xy 204.47 80.01) (xy 207.01 80.01))
+    (stroke (width 0) (type default))
+  )
   (wire (pts (xy 40.64 72.39) (xy 45.72 72.39))
     (stroke (width 0) (type default))
   )
-  (wire (pts (xy 193.04 80.01) (xy 195.58 80.01))
+  (wire (pts (xy 190.5 80.01) (xy 195.58 80.01))
     (stroke (width 0) (type default))
   )
@@
   )
   (wire (pts (xy 146.05 77.47) (xy 143.51 77.47))
-    (stroke (width 0) (type default))
-  )
-  (wire (pts (xy 193.04 60.96) (xy 185.42 60.96))
     (stroke (width 0) (type default))
   )
@@
     (stroke (width 0) (type default))
   )
-  (wire (pts (xy 193.04 80.01) (xy 193.04 60.96))
-    (stroke (width 0) (type default))
-  )

Commit message: Update part 3
Parts:
- removed D1: D, symbol Device:D
- removed R10, R13, R7, R8, R9: R, symbol Device:R
- removed RV1: 1k, symbol Device:R_Potentiometer
- removed U4, U6: LM324, symbol Amplifier_Operational:LM324
- removed U5: LM339, symbol Comparator:LM339
- added D?: 1N4148, symbol Device:D
- added MK?: Microphone_Crystal, symbol Device:Microphone_Crystal
- added R?: 1K, symbol Device:R
- added R?: 10K, symbol Device:R
- added R?: 2K2, symbol Device:R
- added R?: 12K, symbol Device:R
- added R?: 470K, symbol Device:R
- added U? (x3): LM324, symbol Amplifier_Operational:LM324
- C1: value .01u -> 0.01uF
- C1: value .01u -> 4.7uF
- C1: value .01u -> 22uF
- D3: value D -> 1N4148
- R15: value R -> 1K
Connections:
- net GND: now also C1.1, MK?.1 (-), R?.1, R?.2, R?.2, U?.13 (-); no longer C1.2, U7.4 (-)
- net at C1.2, R14.2: now also U?.12 (+)
- net at C1.2, D3.1 (K), R15.2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: no longer R14.1
- net +10V: now reaches R11.2
- net +10V: now also R?.2
- net at D3.2 (A): now also R14.1, U?.14
- new net: R?.1, R?.2, U7.4 (-)
- new net: MK?.2 (+), R?.1, U?.3 (+)
- new net: C1.2, D?.1 (K), R?.2
- new net: R?.1, R?.1, U?.2 (-)
- new net: D?.2 (A), U?.1
Other:
- note added: "G = 40V/V output is 4Vpk Too high is 5V Too low is 3V"
- note added: "On proper bounce, output is 100mVpk Too high is 125mV Too low is 75mV"
- note removed: "Peak Detector"
- note removed: "RC time constant determines "cooldown" of when to flash"
- note removed: "hysteresis"
- moved on the sheet: D4, R11, U7A

Commit message: output stage
Parts:
- removed C1: 0.01uF, symbol Device:C
- removed D3: 1N4148, symbol Device:D
- removed D4: LED, symbol Device:LED
- removed R11: 100, symbol Device:R
- removed R14: R, symbol Device:R
- removed U?: LM324, symbol Amplifier_Operational:LM324
- added D303: LED, symbol Device:LED
- added Q301: NMOS, symbol Simulation_SPICE:NMOS
- added R308: 4.7k, symbol Device:R
- added R309: 100, symbol Device:R
- C1: value 22uF -> .022u
Connections:
- net +10V: now also D303.2 (A), R308.2
- net GND: now also Q301.3 (S)
- net at U7.2: now also Q301.2 (G), R308.1
- new net: D303.1 (K), R309.2
- new net: Q301.1 (D), R309.1

Commit message: Complete first revision lab 3 Schematic
Parts:
- removed U7: LM339, symbol Comparator:LM339
- removed U? (x2): LM324, symbol Amplifier_Operational:LM324
- added C303: 0.01uF, symbol Device:C
- added R309: R, symbol Device:R
- added R312, R313, R314: ??, symbol Device:R
- added R315: 2K2, symbol Device:R
- added U301: LM324, symbol Amplifier_Operational:LM324
- added U302: LM339, symbol Comparator:LM339
- C1: value 4.7uF -> 0.47uF
- C1: value .022u -> 0.022uF
- R319: renamed from R308; value 4.7k -> 4K7
- gave numbers to parts that had none: 7
- renumbered D303 to D304, R15 to R316, R309 to R320
Connections:
- net +10V: now also R312.2, R315.2, U301.4 (V+)
- net GND: now also R309.2, R313.1, U301.11 (V-)
- net at R317.1, R318.2: now also U302.6 (-)
- net at Q301.2 (G), R319.1: now also U302.1
- net at MK301.2 (+), R308.1: now also U301.3 (+)
- net at C1.2, D303.1 (K), R311.2: now also U302.4 (-)
- net at R310.1, R311.1: now also U301.6 (-)
- net at D303.2 (A): now also U301.7
- net at C1.2, R316.2: now also U301.8, U301.9 (-), U302.7 (+)
- new net: R312.1, R313.2, R314.1, U302.5 (+)
- new net: R314.2, R315.1, U301.10 (+), U302.2
- new net: C303.1, U301.1, U301.2 (-)
- new net: C303.2, R309.1, U301.5 (+)
Other:
- note added: "G = 40V/V output is 5Vpk Too low is 3V"
- note added: "High-pass fc = ????"
- note added: "On proper bounce, output is 125mVpk Too low is 75mV"
- note removed: "G = 40V/V output is 4Vpk Too high is 5V Too low is 3V"
- note removed: "On proper bounce, output is 100mVpk Too high is 125mV Too low is 75mV"
- moved on the sheet: C1, D303, D304, MK301, Q301, R308, R310, R311, R316, R317, R318, R319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

Commit message: final lab3
Parts:
- removed C1: 0.47uF, symbol Device:C
- removed C1: 0.022uF, symbol Device:C
- removed Q301: NMOS, symbol Simulation_SPICE:NMOS
- removed R318: 2K2, symbol Device:R
- removed R319: 4K7, symbol Device:R
- removed R320: 100, symbol Device:R
- removed unit 2 of U302
- added C1: 10u, symbol Device:C
- added C1: 10n, symbol Device:C
- added Q301: NPN, symbol Simulation_SPICE:NPN
- added R325: 10k, symbol Device:R
- added U304: LM324, symbol Amplifier_Operational:LM324
- added U305: 4047, symbol 4xxx:4047
- R310: value 12K -> 10k
- R311: value 470K -> 390k
- R312: value ?? -> 82k
- R313: value ?? -> 20k
- R314: value ?? -> 10k
- R316: value 1K -> 820k
- R317: value 1K -> 100
Connections:
- net +10V: now also R317.1, U305.14 (VDD), U305.4 (~{ASTABLE}), U305.8 (+TRIGGER); no longer D304.2 (A), R317.2
- net GND: now also C1.1, Q301.3 (E), R325.2, U305.12 (RETRIGGER), U305.5 (ASTABLE), U305.7 (VSS), U305.9 (EXT_RESET); no longer R316.1
- net at D304.1 (K): now also Q301.1 (C)
- net at D303.1 (K), U302.4 (-): now also C1.2, R325.1, U304.6 (-); no longer R311.2
- net at U301.8, U301.9 (-): now also U305.6 (-TRIGGER); no longer R316.2
- net at U301.7: now also R311.2, U304.5 (+); no longer D303.2 (A)
- new net: C1.2, U305.1 (C)
- new net: Q301.2 (B), U305.11 (~{Q})
- new net: R316.1, U305.2 (R)
- new net: C1.1, R316.2, U305.3 (RC_COMMON)
- new net: D303.2 (A), U304.7
- new net: D304.2 (A), R317.2
- no-connect marks 0 -> 2
Other:
- moved on the sheet: C303, MK301, R308, R309, R310, R311, R312, R313, R314, R315, U301A, U301B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

Commit message: Finalize Lab 3 Post-Recitation
Parts:
- removed C303: 0.01uF, symbol Device:C
- removed R309: R, symbol Device:R
- removed R313: 20k, symbol Device:R
- removed unit 3 of U301
- added RV?: 20K, symbol Device:R_Potentiometer
- C1: value 10n -> 10nF
- R316: value 820k -> 820K
Connections:
- net GND: now also RV?.3
- net at R314.1, U302.5 (+): now also RV?.2; no longer R312.1
- net at R314.2, R315.1, U302.2: now also U305.6 (-TRIGGER)
- net at U301.1, U301.2 (-): now also U301.5 (+)
- net at U305.2 (R): now also R316.2; no longer R316.1
- net at C1.1, U305.3 (RC_COMMON): now also R316.1; no longer R316.2
- new net: R312.1, RV?.1
Other:
- note added: "Active Peak Detector"
- note added: "Gain"
- note added: "Input"
- note added: "Inverting Comparator"
- note added: "Monostable Multivibrator"
- note removed: "High-pass fc = ????"
- moved on the sheet: C1, D303, D304, MK301, Q301, R308, R310, R311, R312, R314, R315, R316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
