File: Lab_03/KiCad/Lab03.kicad_sch (KiCad schematic)
At the start: 0 parts

Commit message: Start Problem 2
Other:
- added sheet Part 2 (L03P02.kicad_sch)
Changed lines of the file:
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@@
+    (instances
+      (project "Lab03"
+        (path "/0f3a9aa4-582a-427a-a342-2cdf273d26d7" (page "1"))
+      )
+    )
+  )
+  (sheet (at 104.14 104.14) (size 43.18 25.4) (fields_autoplaced)
+    (stroke (width 0.1524) (type solid))
+    (fill (color 0 0 0 0.0000))
+    (property "Sheetname" "Part 2" (at 104.14 103.4284 0)
+      (effects (font (size 1.27 1.27)) (justify left bottom))
+    )
+    (property "Sheetfile" "L03P02.kicad_sch" (at 104.14 130.1246 0)
+      (effects (font (size 1.27 1.27)) (justify left top))
+    )
     (instances
       (project "Lab03"
@@
   )
   (sheet_instances
-    (path "/" (page "1"))
+    (path "/" (page "0"))
   )
 )

Commit message: 1 done
Other:
- added sheet Part 3 (part3.kicad_sch)
Changed lines of the file:
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@@
 (kicad_sch (version 20230121) (generator eeschema)
   (paper "A4")
+  (sheet (at 158.75 104.14) (size 41.91 25.4) (fields_autoplaced)
+    (stroke (width 0.1524) (type solid))
+    (fill (color 0 0 0 0.0000))
+    (property "Sheetname" "Part 3" (at 158.75 103.4284 0)
+      (effects (font (size 1.27 1.27)) (justify left bottom))
+    )
+    (property "Sheetfile" "part3.kicad_sch" (at 158.75 130.1246 0)
+      (effects (font (size 1.27 1.27)) (justify left top))
+    )
+    (property "Field2" "" (at 158.75 104.14 0)
+      (effects (font (size 1.27 1.27)) hide)
+    )
+    (instances
+      (project "Lab03"
+        (path "/0f3a9aa4-582a-427a-a342-2cdf273d26d7" (page "4"))
+      )
+    )
+  )
   (sheet (at 104.14 64.77) (size 43.18 26.67) (fields_autoplaced)
     (stroke (width 0.1524) (type solid))

Commit message: Update earlier parts of lab03
Other:
- added sheet Extras (L03_Extras.kicad_sch)
Changed lines of the file:
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@@
 (kicad_sch (version 20230121) (generator eeschema)
   (paper "A4")
+  (sheet (at 22.86 152.4) (size 63.5 36.83) (fields_autoplaced)
+    (stroke (width 0.1524) (type solid))
+    (fill (color 0 0 0 0.0000))
+    (property "Sheetname" "Extras" (at 22.86 151.6884 0)
+      (effects (font (size 1.27 1.27)) (justify left bottom))
+    )
+    (property "Sheetfile" "L03_Extras.kicad_sch" (at 22.86 189.8146 0)
+      (effects (font (size 1.27 1.27)) (justify left top))
+    )
+    (instances
+      (project "Lab03"
+        (path "/0f3a9aa4-582a-427a-a342-2cdf273d26d7" (page "5"))
+      )
+    )
+  )
   (sheet (at 158.75 104.14) (size 41.91 25.4) (fields_autoplaced)
     (stroke (width 0.1524) (type solid))
@@
     (instances
       (project "Lab03"
-        (path "/0f3a9aa4-582a-427a-a342-2cdf273d26d7" (page "4"))
+        (path "/0f3a9aa4-582a-427a-a342-2cdf273d26d7" (page "3"))
       )
     )
