File: Lab_03/KiCad/L03P02.kicad_sch (KiCad schematic)
At the start: 3 parts

Commit message: 1 done
Parts:
- added C1: .01u, symbol Device:C
- added D1: D, symbol Device:D
- added U3: LM741, symbol Amplifier_Operational:LM741
Connections:
- net GND: now also C1.2
- new net: D1.2 (A), U3.6
- new net +15V: U3.7 (V+)
- new net -15V: U3.4 (V-)
- new net Vin_B: U3.3 (+)
- new net Vout_B: C1.1, D1.1 (K), U3.2 (-)
- no-connect marks 0 -> 2
Changed lines of the file:
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@@
 (kicad_sch (version 20230121) (generator eeschema)
   (paper "A4")
+  (junction (at 177.8 45.72) (diameter 0) (color 0 0 0 0)
+  )
+  (junction (at 181.61 45.72) (diameter 0) (color 0 0 0 0)
+  )
   (junction (at 67.31 46.99) (diameter 0) (color 0 0 0 0)
   )
+  (no_connect (at 161.29 53.34))
+  (no_connect (at 163.83 53.34))
+  (wire (pts (xy 151.13 62.23) (xy 151.13 48.26))
+    (stroke (width 0) (type default))
+  )
+  (wire (pts (xy 177.8 45.72) (xy 181.61 45.72))
+    (stroke (width 0) (type default))
+  )
   (wire (pts (xy 53.34 46.99) (xy 57.15 46.99))
     (stroke (width 0) (type default))
@@
     (stroke (width 0) (type default))
   )
+  (wire (pts (xy 151.13 48.26) (xy 153.67 48.26))
+    (stroke (width 0) (type default))
+  )
+  (wire (pts (xy 148.59 43.18) (xy 153.67 43.18))
+    (stroke (width 0) (type default))
+  )
   (wire (pts (xy 67.31 46.99) (xy 67.31 50.8))
     (stroke (width 0) (type default))
   )
+  (wire (pts (xy 168.91 45.72) (xy 170.18 45.72))
+    (stroke (width 0) (type default))
+  )
+  (wire (pts (xy 177.8 45.72) (xy 177.8 62.23))
+    (stroke (width 0) (type default))
+  )
+  (wire (pts (xy 181.61 45.72) (xy 185.42 45.72))
+    (stroke (width 0) (type default))
+  )
   (wire (pts (xy 40.64 46.99) (xy 45.72 46.99))
     (stroke (width 0) (type default))
   )
+  (wire (pts (xy 158.75 36.83) (xy 158.75 38.1))
+    (stroke (width 0) (type default))
+  )
   (wire (pts (xy 67.31 46.99) (xy 77.47 46.99))
     (stroke (width 0) (type default))
@@
     (stroke (width 0) (type default))
   )
+  (wire (pts (xy 181.61 53.34) (xy 181.61 54.61))
+    (stroke (width 0) (type default))
+  )
+  (wire (pts (xy 177.8 62.23) (xy 151.13 62.23))
+    (stroke (width 0) (type default))
+  )
+  (wire (pts (xy 158.75 53.34) (xy 158.75 54.61))
+    (stroke (width 0) (type default))
+  )
   (rectangle (start 27.94 26.67) (end 91.44 73.66)
     (stroke (width 0) (type default))
     (fill (type none))
+  )
+  (text "2A" (at 127 33.02 0)
+    (effects (font (size 5.08 5.08) (thickness 1.016) bold) (justify left bottom))
   )
   (text "2A" (at 27.94 34.29 0)
     (effects (font (size 5.08 5.08) (thickness 1.016) bold) (justify left bottom))
   )
+  (hierarchical_label "Vout_B" (shape output) (at 185.42 45.72 0) (fields_autoplaced)
+    (effects (font (size 1.27 1.27)) (justify left))
+  )
+  (hierarchical_label "Vin_B" (shape input) (at 148.59 43.18 180) (fields_autoplaced)
+    (effects (font (size 1.27 1.27)) (justify right))
+  )
   (hierarchical_label "Vout_A" (shape output) (at 77.47 46.99 0) (fields_autoplaced)
     (effects (font (size 1.27 1.27)) (justify left))
@@
   (hierarchical_label "Vin_A" (shape input) (at 40.64 46.99 180) (fields_autoplaced)
     (effects (font (size 1.27 1.27)) (justify right))
+  )
+  (symbol (lib_id "power:GND") (at 181.61 54.61 0) (unit 1)
+    (in_bom yes) (on_board yes) (dnp no) (fields_autoplaced)
+    (property "Reference" "#PWR07" (at 181.61 60.96 0)
+      (effects (font (size 1.27 1.27)) hide)
+    )
+    (property "Value" "GND" (at 181.61 59.69 0)
+      (effects (font (size 1.27 1.27)))
+    )
+    (property "Footprint" "" (at 181.61 54.61 0)
+      (effects (font (size 1.27 1.27)) hide)
+    )
+    (property "Datasheet" "" (at 181.61 54.61 0)
+      (effects (font (size 1.27 1.27)) hide)
+    )
+    (pin "1")
+    (instances
+      (project "Lab03"
+        (path "/0f3a9aa4-582a-427a-a342-2cdf273d26d7/f6b0de55-6a15-45d1-9616-af32507e700a"
+          (reference "#PWR07") (unit 1)
+        )
+      )
+    )
+  )
+  (symbol (lib_id "Device:D") (at 173.99 45.72 180) (unit 1)
+    (in_bom yes) (on_board yes) (dnp no) (fields_autoplaced)
+    (property "Reference" "D1" (at 173.99 39.37 0)
+      (effects (font (size 1.27 1.27)))
+    )
+    (property "Value" "D" (at 173.99 41.91 0)
+      (effects (font (size 1.27 1.27)))
+    )
+    (property "Footprint" "" (at 173.99 45.72 0)
+      (effects (font (size 1.27 1.27)) hide)
+    )
+    (property "Datasheet" "~" (at 173.99 45.72 0)
+      (effects (font (size 1.27 1.27)) hide)
+    )
+    (property "Sim.Device" "D" (at 173.99 45.72 0)
+      (effects (font (size 1.27 1.27)) hide)
+    )
+    (property "Sim.Pins" "1=K 2=A" (at 173.99 45.72 0)
+      (effects (font (size 1.27 1.27)) hide)
+    )
+    (pin "1")
+    (pin "2")
+    (instances
+      (project "Lab03"
+        (path "/0f3a9aa4-582a-427a-a342-2cdf273d26d7/f6b0de55-6a15-45d1-9616-af32507e700a"
+          (reference "D1") (unit 1)
+        )
+      )
+    )
   )
   (symbol (lib_id "Device:R") (at 49.53 46.99 90) (unit 1)
@@
     )
   )
+  (symbol (lib_id "power:+15V") (at 158.75 36.83 0) (unit 1)
+    (in_bom yes) (on_board yes) (dnp no) (fields_autoplaced)
+    (property "Reference" "#PWR09" (at 158.75 40.64 0)
+      (effects (font (size 1.27 1.27)) hide)
+    )
+    (property "Value" "+15V" (at 158.75 31.75 0)
+      (effects (font (size 1.27 1.27)))
+    )
+    (property "Footprint" "" (at 158.75 36.83 0)
+      (effects (font (size 1.27 1.27)) hide)
+    )
+    (property "Datasheet" "" (at 158.75 36.83 0)
+      (effects (font (size 1.27 1.27)) hide)
+    )
+    (pin "1")
+    (instances
+      (project "Lab03"
+        (path "/0f3a9aa4-582a-427a-a342-2cdf273d26d7/f6b0de55-6a15-45d1-9616-af32507e700a"
+          (reference "#PWR09") (unit 1)
+        )
+      )
+    )
+  )
+  (symbol (lib_id "power:-15V") (at 158.75 54.61 180) (unit 1)
+    (in_bom yes) (on_board yes) (dnp no) (fields_autoplaced)
+    (property "Reference" "#PWR010" (at 158.75 57.15 0)
+      (effects (font (size 1.27 1.27)) hide)
+    )
+    (property "Value" "-15V" (at 158.75 59.69 0)
+      (effects (font (size 1.27 1.27)))
+    )
+    (property "Footprint" "" (at 158.75 54.61 0)
+      (effects (font (size 1.27 1.27)) hide)
+    )
+    (property "Datasheet" "" (at 158.75 54.61 0)
+      (effects (font (size 1.27 1.27)) hide)
+    )
+    (pin "1")
+    (instances
+      (project "Lab03"
+        (path "/0f3a9aa4-582a-427a-a342-2cdf273d26d7/f6b0de55-6a15-45d1-9616-af32507e700a"
+          (reference "#PWR010") (unit 1)
+        )
+      )
+    )
+  )
+  (symbol (lib_id "Amplifier_Operational:LM741") (at 161.29 45.72 0) (unit 1)
+    (in_bom yes) (on_board yes) (dnp no)
+    (property "Reference" "U3" (at 171.45 41.5291 0)
+      (effects (font (size 1.27 1.27)))
+    )
+    (property "Value" "LM741" (at 167.64 48.26 0)
+      (effects (font (size 1.27 1.27)))
+    )
+    (property "Footprint" "" (at 162.56 44.45 0)
+      (effects (font (size 1.27 1.27)) hide)
+    )
+    (property "Datasheet" "http://www.ti.com/lit/ds/symlink/lm741.pdf" (at 165.1 41.91 0)
+      (effects (font (size 1.27 1.27)) hide)
+    )
+    (pin "7")
+    (pin "3")
+    (pin "6")
+    (pin "2")
+    (pin "1")
+    (pin "4")
+    (pin "8")
+    (pin "5")
+    (instances
+      (project "Lab03"
+        (path "/0f3a9aa4-582a-427a-a342-2cdf273d26d7/f6b0de55-6a15-45d1-9616-af32507e700a"
+          (reference "U3") (unit 1)
+        )
+      )
+    )
+  )
   (symbol (lib_id "power:GND") (at 67.31 59.69 0) (unit 1)
     (in_bom yes) (on_board yes) (dnp no)
@@
         )
       )
+    )
+  )
+  (symbol (lib_id "Device:C") (at 181.61 49.53 0) (unit 1)
+    (in_bom yes) (on_board yes) (dnp no) (fields_autoplaced)
+    (property "Reference" "C1" (at 185.42 48.26 0)
+      (effects (font (size 1.27 1.27)) (justify left))
+    )
+    (property "Value" ".01u" (at 185.42 50.8 0)
+      (effects (font (size 1.27 1.27)) (justify left))
+    )
+    (property "Footprint" "" (at 182.5752 53.34 0)
+      (effects (font (size 1.27 1.27)) hide)
+    )
+    (property "Datasheet" "~" (at 181.61 49.53 0)
+      (effects (font (size 1.27 1.27)) hide)
+    )
+    (pin "1")
+    (pin "2")
+    (instances
+      (project "Lab03"
+        (path "/0f3a9aa4-582a-427a-a342-2cdf273d26d7/f6b0de55-6a15-45d1-9616-af32507e700a"
+          (reference "C1") (unit 1)
+        )
+      )

Commit message: Finish Schematics & Scope traces through part 2
Other:
- note added: "2B"
Changed lines of the file:
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@@
     (stroke (width 0) (type default))
+  )
+  (rectangle (start 127 25.4) (end 195.58 72.39)
+    (stroke (width 0) (type default))
+    (fill (type none))
   )
   (rectangle (start 27.94 26.67) (end 91.44 73.66)
@@
     (fill (type none))
   )
-  (text "2A" (at 127 33.02 0)
+  (text "2B" (at 127 33.02 0)
     (effects (font (size 5.08 5.08) (thickness 1.016) bold) (justify left bottom))
   )
@@
   (symbol (lib_id "Amplifier_Operational:LM741") (at 161.29 45.72 0) (unit 1)
     (in_bom yes) (on_board yes) (dnp no)
-    (property "Reference" "U3" (at 171.45 41.5291 0)
+    (property "Reference" "U3" (at 163.83 41.91 0)
       (effects (font (size 1.27 1.27)))
     )
@@
       (effects (font (size 1.27 1.27)) hide)
     )
+    (pin "1")
+    (pin "2")
+    (pin "3")
+    (pin "4")
+    (pin "5")
+    (pin "6")
     (pin "7")
-    (pin "3")
-    (pin "6")
-    (pin "2")
-    (pin "1")
-    (pin "4")
     (pin "8")
-    (pin "5")
     (instances
       (project "Lab03"

Commit message: Update earlier parts of lab03
Parts:
- renumbered C201 to C301, C1 to C302, D201 to D301, D1 to D302, R201 to R307, U3 to U303
Changed lines of the file:
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@@
   (symbol (lib_id "power:GND") (at 181.61 54.61 0) (unit 1)
     (in_bom yes) (on_board yes) (dnp no) (fields_autoplaced)
-    (property "Reference" "#PWR07" (at 181.61 60.96 0)
+    (property "Reference" "#PWR0310" (at 181.61 60.96 0)
       (effects (font (size 1.27 1.27)) hide)
     )
@@
       (project "Lab03"
         (path "/0f3a9aa4-582a-427a-a342-2cdf273d26d7/f6b0de55-6a15-45d1-9616-af32507e700a"
-          (reference "#PWR07") (unit 1)
+          (reference "#PWR0310") (unit 1)
         )
       )
@@
   (symbol (lib_id "Device:D") (at 173.99 45.72 180) (unit 1)
     (in_bom yes) (on_board yes) (dnp no) (fields_autoplaced)
-    (property "Reference" "D1" (at 173.99 39.37 0)
+    (property "Reference" "D302" (at 173.99 39.37 0)
       (effects (font (size 1.27 1.27)))
     )
@@
       (project "Lab03"
         (path "/0f3a9aa4-582a-427a-a342-2cdf273d26d7/f6b0de55-6a15-45d1-9616-af32507e700a"
-          (reference "D1") (unit 1)
+          (reference "D302") (unit 1)
         )
       )
@@
   (symbol (lib_id "Device:R") (at 49.53 46.99 90) (unit 1)
     (in_bom yes) (on_board yes) (dnp no)
-    (property "Reference" "R201" (at 49.53 44.45 90)
+    (property "Reference" "R307" (at 49.53 44.45 90)
       (effects (font (size 1.27 1.27)))
     )
@@
       (project "Lab03"
         (path "/0f3a9aa4-582a-427a-a342-2cdf273d26d7/f6b0de55-6a15-45d1-9616-af32507e700a"
-          (reference "R201") (unit 1)
+          (reference "R307") (unit 1)
         )
       )
@@
   (symbol (lib_id "power:+15V") (at 158.75 36.83 0) (unit 1)
     (in_bom yes) (on_board yes) (dnp no) (fields_autoplaced)
-    (property "Reference" "#PWR09" (at 158.75 40.64 0)
+    (property "Reference" "#PWR0308" (at 158.75 40.64 0)
       (effects (font (size 1.27 1.27)) hide)
     )
@@
       (project "Lab03"
         (path "/0f3a9aa4-582a-427a-a342-2cdf273d26d7/f6b0de55-6a15-45d1-9616-af32507e700a"
-          (reference "#PWR09") (unit 1)
+          (reference "#PWR0308") (unit 1)
         )
       )
@@
   (symbol (lib_id "power:-15V") (at 158.75 54.61 180) (unit 1)
     (in_bom yes) (on_board yes) (dnp no) (fields_autoplaced)
-    (property "Reference" "#PWR010" (at 158.75 57.15 0)
+    (property "Reference" "#PWR0309" (at 158.75 57.15 0)
       (effects (font (size 1.27 1.27)) hide)
     )
@@
       (project "Lab03"
         (path "/0f3a9aa4-582a-427a-a342-2cdf273d26d7/f6b0de55-6a15-45d1-9616-af32507e700a"
-          (reference "#PWR010") (unit 1)
+          (reference "#PWR0309") (unit 1)
         )
       )
@@
   (symbol (lib_id "Amplifier_Operational:LM741") (at 161.29 45.72 0) (unit 1)
     (in_bom yes) (on_board yes) (dnp no)
-    (property "Reference" "U3" (at 163.83 41.91 0)
+    (property "Reference" "U303" (at 163.83 41.91 0)
       (effects (font (size 1.27 1.27)))
     )
@@
       (project "Lab03"
         (path "/0f3a9aa4-582a-427a-a342-2cdf273d26d7/f6b0de55-6a15-45d1-9616-af32507e700a"
-          (reference "U3") (unit 1)
+          (reference "U303") (unit 1)
         )
       )
@@
         )
         (path "/0f3a9aa4-582a-427a-a342-2cdf273d26d7/f6b0de55-6a15-45d1-9616-af32507e700a"
-          (reference "#PWR08") (unit 1)
+          (reference "#PWR0307") (unit 1)
         )
       )
@@
   (symbol (lib_id "Device:C") (at 181.61 49.53 0) (unit 1)
     (in_bom yes) (on_board yes) (dnp no) (fields_autoplaced)
-    (property "Reference" "C1" (at 185.42 48.26 0)
+    (property "Reference" "C302" (at 185.42 48.26 0)
       (effects (font (size 1.27 1.27)) (justify left))
     )
@@
       (project "Lab03"
         (path "/0f3a9aa4-582a-427a-a342-2cdf273d26d7/f6b0de55-6a15-45d1-9616-af32507e700a"
-          (reference "C1") (unit 1)
+          (reference "C302") (unit 1)
         )
       )
@@
   (symbol (lib_id "Diode:1N4148") (at 60.96 46.99 180) (unit 1)
     (in_bom yes) (on_board yes) (dnp no) (fields_autoplaced)
-    (property "Reference" "D201" (at 60.96 40.64 0)
+    (property "Reference" "D301" (at 60.96 40.64 0)
       (effects (font (size 1.27 1.27)))
     )
@@
       (project "Lab03"
         (path "/0f3a9aa4-582a-427a-a342-2cdf273d26d7/f6b0de55-6a15-45d1-9616-af32507e700a"
-          (reference "D201") (unit 1)
+          (reference "D301") (unit 1)
         )
       )
@@
   (symbol (lib_id "Device:C") (at 67.31 54.61 0) (unit 1)
     (in_bom yes) (on_board yes) (dnp no)
-    (property "Reference" "C201" (at 68.58 52.07 0)
+    (property "Reference" "C301" (at 68.58 52.07 0)
       (effects (font (size 1.27 1.27)) (justify left))
     )
@@
       (project "Lab03"
         (path "/0f3a9aa4-582a-427a-a342-2cdf273d26d7/f6b0de55-6a15-45d1-9616-af32507e700a"
-          (reference "C201") (unit 1)
-        )
-      )
+          (reference "C301") (unit 1)
+        )
+      )

Commit message: Finalize Lab 3 Post-Recitation
Parts:
- removed D301: 1N4148, Diode_THT:D_DO-35_SOD27_P7.62mm_Horizontal, symbol Diode:1N4148
- added D?: 1N5819, Diode_THT:D_DO-41_SOD81_P10.16mm_Horizontal, symbol Diode:1N5819
Connections:
- net Vout_A: now also D?.1 (K)
- net at R307.2: now also D?.2 (A)
Changed lines of the file:
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@@
+    )
+  )
+  (symbol (lib_id "Diode:1N5819") (at 60.96 46.99 180) (unit 1)
+    (in_bom yes) (on_board yes) (dnp no) (fields_autoplaced)
+    (property "Reference" "D?" (at 61.2775 40.64 0)
+      (effects (font (size 1.27 1.27)))
+    )
+    (property "Value" "1N5819" (at 61.2775 43.18 0)
+      (effects (font (size 1.27 1.27)))
+    )
+    (property "Footprint" "Diode_THT:D_DO-41_SOD81_P10.16mm_Horizontal" (at 60.96 42.545 0)
+      (effects (font (size 1.27 1.27)) hide)
+    )
+    (property "Datasheet" "http://www.vishay.com/docs/88525/1n5817.pdf" (at 60.96 46.99 0)
+      (effects (font (size 1.27 1.27)) hide)
+    )
+    (pin "1")
+    (pin "2")
+    (instances
+      (project "Lab03"
+        (path "/0f3a9aa4-582a-427a-a342-2cdf273d26d7/f6b0de55-6a15-45d1-9616-af32507e700a"
+          (reference "D?") (unit 1)
+        )
+      )
     )
   )
@@
         )
       )
-    )
-  )
-  (symbol (lib_id "Diode:1N4148") (at 60.96 46.99 180) (unit 1)
-    (in_bom yes) (on_board yes) (dnp no) (fields_autoplaced)
-    (property "Reference" "D301" (at 60.96 40.64 0)
-      (effects (font (size 1.27 1.27)))
-    )
-    (property "Value" "1N4148" (at 60.96 43.18 0)
-      (effects (font (size 1.27 1.27)))
-    )
-    (property "Footprint" "Diode_THT:D_DO-35_SOD27_P7.62mm_Horizontal" (at 60.96 46.99 0)
-      (effects (font (size 1.27 1.27)) hide)
-    )
-    (property "Datasheet" "https://assets.nexperia.com/documents/data-sheet/1N4148_1N4448.pdf" (at 60.96 46.99 0)
-      (effects (font (size 1.27 1.27)) hide)
-    )
-    (property "Sim.Device" "D" (at 60.96 46.99 0)
-      (effects (font (size 1.27 1.27)) hide)
-    )
-    (property "Sim.Pins" "1=K 2=A" (at 60.96 46.99 0)
-      (effects (font (size 1.27 1.27)) hide)
-    )
-    (pin "1")
-    (pin "2")
-    (instances
-      (project "Lab03"
-        (path "/0f3a9aa4-582a-427a-a342-2cdf273d26d7/f6b0de55-6a15-45d1-9616-af32507e700a"
-          (reference "D301") (unit 1)
-        )
-      )
