File: Lab_04/Lab04.kicad_sch (KiCad schematic)
At the start: 0 parts

Commit message: 123 done
Other:
- added sheet Part2 (part2.kicad_sch)
- added sheet Part3 (part3.kicad_sch)
- added sheet Part4 (part4.kicad_sch)
Changed lines of the file:
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@@
+    )
+  )
+  (sheet (at 175.26 43.18) (size 36.83 25.4) (fields_autoplaced)
+    (stroke (width 0.1524) (type solid))
+    (fill (color 0 0 0 0.0000))
+    (property "Sheetname" "Part3" (at 175.26 42.4684 0)
+      (effects (font (size 1.27 1.27)) (justify left bottom))
+    )
+    (property "Sheetfile" "part3.kicad_sch" (at 175.26 69.1646 0)
+      (effects (font (size 1.27 1.27)) (justify left top))
+    )
+    (property "Field2" "" (at 175.26 43.18 0)
+      (effects (font (size 1.27 1.27)) hide)
+    )
+    (instances
+      (project "Lab04"
+        (path "/d11ac0ed-f6df-48cb-8771-3e619bea6e62" (page "4"))
+      )
+    )
+  )
+  (sheet (at 223.52 43.18) (size 36.83 25.4) (fields_autoplaced)
+    (stroke (width 0.1524) (type solid))
+    (fill (color 0 0 0 0.0000))
+    (property "Sheetname" "Part4" (at 223.52 42.4684 0)
+      (effects (font (size 1.27 1.27)) (justify left bottom))
+    )
+    (property "Sheetfile" "part4.kicad_sch" (at 223.52 69.1646 0)
+      (effects (font (size 1.27 1.27)) (justify left top))
+    )
+    (property "Field2" "" (at 223.52 43.18 0)
+      (effects (font (size 1.27 1.27)) hide)
+    )
+    (instances
+      (project "Lab04"
+        (path "/d11ac0ed-f6df-48cb-8771-3e619bea6e62" (page "5"))
+      )
+    )
+  )
+  (sheet (at 123.19 43.18) (size 36.83 25.4) (fields_autoplaced)
+    (stroke (width 0.1524) (type solid))
+    (fill (color 0 0 0 0.0000))
+    (property "Sheetname" "Part2" (at 123.19 42.4684 0)
+      (effects (font (size 1.27 1.27)) (justify left bottom))
+    )
+    (property "Sheetfile" "part2.kicad_sch" (at 123.19 69.1646 0)
+      (effects (font (size 1.27 1.27)) (justify left top))
+    )
+    (property "Field2" "" (at 123.19 43.18 0)
+      (effects (font (size 1.27 1.27)) hide)
+    )
+    (instances
+      (project "Lab04"
+        (path "/d11ac0ed-f6df-48cb-8771-3e619bea6e62" (page "3"))
+      )
     )
   )
