File: Lab_05/KiCad_Files/Lab05.kicad_sch (KiCad schematic)
At the start: 0 parts

Commit message: Continue Lab 5
Other:
- company: (none) -> Jim Horwitz & Mark Vaughn, Jork Incorporated
Changed lines of the file:
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@@
 (kicad_sch (version 20230121) (generator eeschema)
   (paper "A4")
+  (title_block
+    (date "2024-02-17")
+    (company "Jim Horwitz & Mark Vaughn, Jork Incorporated")
+  )
   (sheet (at 173.99 53.34) (size 38.1 24.13) (fields_autoplaced)
     (stroke (width 0.1524) (type solid))
