File: Lab_06/Kicad_Files/02_SqTriOsc.kicad_sch (KiCad schematic)
At the start: 0 parts

Commit message: Begin Saturday Schematic
Parts:
- added C?: 10C, symbol Device:C
- added C?: C, symbol Device:C
- added D? (x4): ~, symbol Lab06:D_45
- added Q?: NPN, symbol Simulation_SPICE:NPN
- added Q?: PNP, symbol Simulation_SPICE:PNP
- added R?: 22K, symbol Device:R
- added R?: 10K, symbol Device:R
- added R? (x2): R, symbol Device:R
- added SW?: RANGE, symbol Lab06:SW_SPDT
- added U? (x5): LM324A, symbol Amplifier_Operational:LM324A
Connections:
- new net: D?.1 (K), D?.1 (K), Q?.1 (C)
- new net: Q?.3 (E), R?.1
- new net: C?.1, SW?.1 (A)
- new net: D?.1 (K), D?.2 (A), SW?.2 (B), U?.3 (+)
- new net: C?.1, SW?.3 (C)
- new net: R?.1, R?.1, U?.5 (+)
- new net: D?.2 (A), D?.2 (A), Q?.1 (C)
- new net: Q?.3 (E), R?.2
- new net +15V: R?.1, U?.4 (V+)
- new net -15V: R?.2, U?.11 (V-)
- new net GND: C?.2, C?.2, R?.2
- new net SQUARE_OUT: D?.1 (K), D?.2 (A), R?.2, U?.7
- new net TRIANGLE_OUT: U?.1, U?.2 (-), U?.6 (-)

Commit message: Continue Lab 6 Saturday Schematic
Parts:
- added R201, R202, R203, R204, R205, R206: R, symbol Device:R
- added RV201: 10K, symbol Device:R_Potentiometer
- added RV202: 10K, symbol Device:R_Potentiometer_Trim
- gave numbers to parts that had none: 14
Connections:
- net +15V: now also RV201.1, RV202.1
- net GND: now also U201.12 (+), R204.2, RV201.3, RV202.3
- net at Q202.2 (B): now also U201.14, R205.2
- net at U201.13 (-): now also R202.2, R203.2, R205.1
- net at U201.10 (+): now also R201.2, R203.1
- net at U201.8: now also Q201.2 (B), R206.2
- net at U201.9 (-): now also R204.1, R206.1
- new net: R201.1, RV201.2
- new net: R202.1, RV202.2
Other:
- note added: "Close to -15+VBE"
- note added: "Close to 15-VBE"
- note added: "Frequency Adjust"
- note added: "Range"
- note added: "Symmetry Trim"
- title: (none) -> Diode Bridge Square/Triangle Oscillator
- moved on the sheet: C201, C202, D201, D202, D203, D204, Q201, Q202, R207, R208, R209, R210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

Commit message: Finish Saturday Schematic
Parts:
- added D205, D206, D207, D208: D, symbol Device:D
- added Q203, Q204: NPN, symbol Simulation_SPICE:NPN
- added R209, R214: R, symbol Device:R
- added R210, R215: 10K, symbol Device:R
- added R213: 47K, symbol Device:R
- R211: renamed from R209; value 22K -> 3K3
- R212: renamed from R210; value 10K -> 22K
Connections:
- net GATE_IN: now also R209.1, R214.1
- net GND: now also D206.1 (K), D208.2 (A), Q203.3 (E), Q204.3 (E), R210.2, R215.2
- net SQUARE_OUT: now also D205.2 (A), D207.1 (K), Q204.1 (C), R213.2; no longer D201.1 (K), D202.2 (A), R212.2, U201.7
- net at D203.1 (K), D204.2 (A), SW201.2 (B)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: now also Q203.1 (C)
- new net: Q203.2 (B), R209.2, R210.1
- new net: D205.1 (K), D206.2 (A)
- new net: D207.2 (A), D208.1 (K)
- new net: Q204.2 (B), R214.2, R215.1
- new net: D201.1 (K), D202.2 (A), R212.2, R213.1, U201.7
Other:
- note added: "2Vpk-pk"
- note removed: "Close to -15+VBE"
- note removed: "Close to 15-VBE"
- moved on the sheet: C201, C202, D201, D202, D203, D204, Q201, Q202, R201, R202, R203, R204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
