File: Lab_06/Kicad_Files/03_SinShape.kicad_sch (KiCad schematic)
At the start: 0 parts

Commit message: Finish Saturday Schematic
Parts:
- added D301, D302: D, symbol Device:D
- added R301: 220R, symbol Device:R
Connections:
- net SINE_OUT: now also D301.2 (A), D302.1 (K), R301.2
- net TRIANGLE_IN: now also R301.1
- new net GND: D301.1 (K), D302.2 (A)
Other:
- note added: "1.4Vpk-pk"
- note added: "2Vpk-pk"
- title: (none) -> Very Simple Sine Converter
Changed lines of the file:
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@@
 (kicad_sch (version 20230121) (generator eeschema)
-  (paper "A4")
+  (paper "User" 177.8 127)
   (title_block
+    (title "Very Simple Sine Converter")
+    (date "2024-02-24")
+    (rev "0")
     (company "ZAM Industries, LLC")
     (comment 1 "Drawn by: Mark Vaughn")
+    (comment 2 "ALL DIODES 1N4148 UNLESS OTHERWISE NOTED")
+    (comment 3 "ALL BJTS 2N4401/2N4403 UNLESS OTHERWISE NOTED")
   )
-  (hierarchical_label "SINE_OUT" (shape output) (at 215.9 88.9 0) (fields_autoplaced)
+  (junction (at 86.36 63.5) (diameter 0) (color 0 0 0 0)
+  )
+  (junction (at 80.01 50.8) (diameter 0) (color 0 0 0 0)
+  )
+  (junction (at 92.71 50.8) (diameter 0) (color 0 0 0 0)
+  )
+  (wire (pts (xy 92.71 60.96) (xy 92.71 63.5))
+    (stroke (width 0) (type default))
+  )
+  (wire (pts (xy 71.12 50.8) (xy 80.01 50.8))
+    (stroke (width 0) (type default))
+  )
+  (wire (pts (xy 92.71 50.8) (xy 92.71 53.34))
+    (stroke (width 0) (type default))
+  )
+  (wire (pts (xy 86.36 63.5) (xy 92.71 63.5))
+    (stroke (width 0) (type default))
+  )
+  (wire (pts (xy 80.01 60.96) (xy 80.01 63.5))
+    (stroke (width 0) (type default))
+  )
+  (wire (pts (xy 86.36 63.5) (xy 86.36 64.77))
+    (stroke (width 0) (type default))
+  )
+  (wire (pts (xy 80.01 50.8) (xy 92.71 50.8))
+    (stroke (width 0) (type default))
+  )
+  (wire (pts (xy 80.01 63.5) (xy 86.36 63.5))
+    (stroke (width 0) (type default))
+  )
+  (wire (pts (xy 80.01 50.8) (xy 80.01 53.34))
+    (stroke (width 0) (type default))
+  )
+  (wire (pts (xy 54.61 50.8) (xy 63.5 50.8))
+    (stroke (width 0) (type default))
+  )
+  (wire (pts (xy 92.71 50.8) (xy 118.11 50.8))
+    (stroke (width 0) (type default))
+  )
+  (text "2Vpk-pk" (at 52.07 55.88 0)
+    (effects (font (size 1.27 1.27)) (justify right bottom))
+  )
+  (text "1.4Vpk-pk" (at 120.65 55.88 0)
+    (effects (font (size 1.27 1.27)) (justify left bottom))
+  )
+  (hierarchical_label "SINE_OUT" (shape output) (at 118.11 50.8 0) (fields_autoplaced)
     (effects (font (size 2.54 2.54) (thickness 0.508) bold) (justify left))
   )
-  (hierarchical_label "TRIANGLE_IN" (shape input) (at 63.5 88.9 180) (fields_autoplaced)
+  (hierarchical_label "TRIANGLE_IN" (shape input) (at 54.61 50.8 180) (fields_autoplaced)
     (effects (font (size 2.54 2.54) (thickness 0.508) bold) (justify right))
   )
+  (symbol (lib_id "Device:R") (at 67.31 50.8 90) (unit 1)
+    (in_bom yes) (on_board yes) (dnp no)
+    (property "Reference" "R301" (at 67.31 48.26 90)
+      (effects (font (size 1.27 1.27)))
+    )
+    (property "Value" "220R" (at 67.31 50.8 90)
+      (effects (font (size 1.27 1.27)))
+    )
+    (property "Footprint" "" (at 67.31 52.578 90)
+      (effects (font (size 1.27 1.27)) hide)
+    )
+    (property "Datasheet" "~" (at 67.31 50.8 0)
+      (effects (font (size 1.27 1.27)) hide)
+    )
+    (pin "1")
+    (pin "2")
+    (instances
+      (project "Lab06"
+        (path "/37d0ecfa-1973-4a3c-8fc1-f7066c204731/992af115-f2cd-423f-adc5-3d2d5603cc4b"
+          (reference "R301") (unit 1)
+        )
+      )
+    )
+  )
+  (symbol (lib_id "Device:D") (at 80.01 57.15 270) (mirror x) (unit 1)
+    (in_bom yes) (on_board yes) (dnp no)
+    (property "Reference" "D301" (at 77.47 57.15 90)
+      (effects (font (size 1.27 1.27)) (justify right))
+    )
+    (property "Value" "D" (at 77.47 58.42 90)
+      (effects (font (size 1.27 1.27)) (justify right) hide)
+    )
+    (property "Footprint" "" (at 80.01 57.15 0)
+      (effects (font (size 1.27 1.27)) hide)
+    )
+    (property "Datasheet" "~" (at 80.01 57.15 0)
+      (effects (font (size 1.27 1.27)) hide)
+    )
+    (property "Sim.Device" "D" (at 80.01 57.15 0)
+      (effects (font (size 1.27 1.27)) hide)
+    )
+    (property "Sim.Pins" "1=K 2=A" (at 80.01 57.15 0)
+      (effects (font (size 1.27 1.27)) hide)
+    )
+    (pin "1")
+    (pin "2")
+    (instances
+      (project "Lab06"
+        (path "/37d0ecfa-1973-4a3c-8fc1-f7066c204731/992af115-f2cd-423f-adc5-3d2d5603cc4b"
+          (reference "D301") (unit 1)
+        )
+      )
+    )
+  )
+  (symbol (lib_id "power:GND") (at 86.36 64.77 0) (unit 1)
+    (in_bom yes) (on_board yes) (dnp no)
+    (property "Reference" "#PWR0301" (at 86.36 71.12 0)
+      (effects (font (size 1.27 1.27)) hide)
+    )
+    (property "Value" "GND" (at 86.36 68.58 0)
+      (effects (font (size 1.27 1.27)))
+    )
+    (property "Footprint" "" (at 86.36 64.77 0)
+      (effects (font (size 1.27 1.27)) hide)
+    )
+    (property "Datasheet" "" (at 86.36 64.77 0)
+      (effects (font (size 1.27 1.27)) hide)
+    )
+    (pin "1")
+    (instances
+      (project "Lab06"
+        (path "/37d0ecfa-1973-4a3c-8fc1-f7066c204731/992af115-f2cd-423f-adc5-3d2d5603cc4b"
+          (reference "#PWR0301") (unit 1)
+        )
+      )
+    )
+  )
+  (symbol (lib_id "Device:D") (at 92.71 57.15 90) (mirror x) (unit 1)
+    (in_bom yes) (on_board yes) (dnp no)
+    (property "Reference" "D302" (at 95.25 57.15 90)
+      (effects (font (size 1.27 1.27)) (justify right))
+    )
+    (property "Value" "D" (at 95.25 58.42 90)
+      (effects (font (size 1.27 1.27)) (justify right) hide)
+    )
+    (property "Footprint" "" (at 92.71 57.15 0)
+      (effects (font (size 1.27 1.27)) hide)
+    )
+    (property "Datasheet" "~" (at 92.71 57.15 0)
+      (effects (font (size 1.27 1.27)) hide)
+    )
+    (property "Sim.Device" "D" (at 92.71 57.15 0)
+      (effects (font (size 1.27 1.27)) hide)
+    )
+    (property "Sim.Pins" "1=K 2=A" (at 92.71 57.15 0)
+      (effects (font (size 1.27 1.27)) hide)
+    )
+    (pin "1")
+    (pin "2")
+    (instances
+      (project "Lab06"
+        (path "/37d0ecfa-1973-4a3c-8fc1-f7066c204731/992af115-f2cd-423f-adc5-3d2d5603cc4b"
+          (reference "D302") (unit 1)
+        )
+      )
+    )
+  )
 )
