File: Lab_06/Kicad_Files/04_PrimaryDrive.kicad_sch (KiCad schematic)
At the start: 0 parts

Commit message: Continue Lab 6 Saturday Schematic
Changed lines of the file:
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@@
     (comment 1 "Drawn by: Mark Vaughn")
   )
-  (hierarchical_label "Waveform_In" (shape input) (at 53.34 62.23 180) (fields_autoplaced)
-    (effects (font (size 1.27 1.27)) (justify right))
+  (hierarchical_label "WAVEFORM_IN" (shape input) (at 53.34 62.23 180) (fields_autoplaced)
+    (effects (font (size 2.54 2.54) (thickness 0.508) bold) (justify right))
   )
-  (hierarchical_label "Waveform_Out" (shape output) (at 187.96 64.77 0) (fields_autoplaced)
-    (effects (font (size 1.27 1.27)) (justify left))
+  (hierarchical_label "WAVEFORM_OUT" (shape output) (at 187.96 64.77 0) (fields_autoplaced)
+    (effects (font (size 2.54 2.54) (thickness 0.508) bold) (justify left))
   )
 )

Commit message: Finish Saturday Schematic
Parts:
- added Q201: PNP, symbol Simulation_SPICE:PNP
- added Q202: NPN, symbol Simulation_SPICE:NPN
- added R201 (x3): R, symbol Device:R
- added R4: 68K, symbol Device:R
- added R4: 8K2, symbol Device:R
- added RV201: 1K, symbol Device:R_Potentiometer_Trim
- added RV201 (x2): 10K, symbol Device:R_Potentiometer
- added U401: LM324A, symbol Amplifier_Operational:LM324A
Connections:
- net WAVEFORM_IN: now also U401.3 (+)
- net WAVEFORM_OUT: now also Q201.1 (C), Q202.1 (C), U401.13 (-)
- new net: R201.1, U401.8, U401.9 (-)
- new net: R201.1, R201.2, R201.2, U401.6 (-)
- new net: R4.2, RV201.1
- new net: RV201.2, U401.2 (-)
- new net: R4.1, RV201.3
- new net: Q201.2 (B), Q202.2 (B), U401.14
- new net: R201.2, U401.12 (+), U401.7
- new net: R4.1, RV201.1, U401.1
- new net: R201.1, RV201.2
- new net: RV201.2, U401.10 (+)
- new net +15V: Q201.3 (E), RV201.1, U401.4 (V+)
- new net -15V: Q202.3 (E), U401.11 (V-)
- new net GND: R4.2, RV201.3, RV201.3, U401.5 (+)
Other:
- note added: "Amplitude Adjust"
- note added: "Max ampl. Trim"
- note added: "Offset Adjust"
- title: (none) -> Triangle/Square/Sine Output Driver
