File: Lab_06/Kicad_Files/05_PWMcontrol.kicad_sch (KiCad schematic)
At the start: 0 parts

Commit message: Finish Saturday Schematic
Parts:
- added R501: 2K2, symbol Device:R
- added RV201: 100K, symbol Device:R_Potentiometer
- added U501: LM393, symbol Comparator:LM393
Connections:
- net PULSE_OUT: now also R501.2, RV201.1, U501.1
- net TRIANGLE_IN: now also U501.2 (-)
- new net: RV201.2, U501.3 (+)
- new net +15V: R501.1, U501.8 (V+)
- new net GND: RV201.3, U501.4 (V-)
- no-connect marks 0 -> 3
Other:
- note added: "0V to 13.5V"
- note added: "Pulse Width Adjust"
- title: (none) -> Triangle to Pulse Converter
