File: Lab_06/Kicad_Files/06_PulseDrive.kicad_sch (KiCad schematic)
At the start: 0 parts

Commit message: Continue Lab 6 Saturday Schematic
Other:
- company: (none) -> ZAM Industries, LLC
Changed lines of the file:
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@@
 (kicad_sch (version 20230121) (generator eeschema)
   (paper "A4")
+  (title_block
+    (company "ZAM Industries, LLC")
+  )
+  (hierarchical_label "PULSE_OUT" (shape output) (at 228.6 88.9 0) (fields_autoplaced)
+    (effects (font (size 2.54 2.54) bold) (justify left))
+  )
+  (hierarchical_label "PULSE_IN" (shape input) (at 62.23 88.9 180) (fields_autoplaced)
+    (effects (font (size 2.54 2.54) bold) (justify right))
+  )
 )

Commit message: Finish Saturday Schematic
Parts:
- added C601: 1000pF, symbol Device:C
- added Q201: PNP, symbol Simulation_SPICE:PNP
- added Q202, Q601: NPN, symbol Simulation_SPICE:NPN
- added R601: 1K, symbol Device:R
- added R602: 220R, symbol Device:R
- added RV201: 1K, symbol Device:R_Potentiometer
Connections:
- net PULSE_IN: now also C601.1, R601.1
- net PULSE_OUT: now also Q201.1 (C), Q202.1 (C)
- new net: Q201.2 (B), Q202.2 (B), Q601.1 (C), RV201.2
- new net: C601.2, Q601.2 (B), R601.2
- new net: R602.2, RV201.1
- new net +15V: Q201.3 (E), R602.1
- new net -15V: Q202.3 (E)
- new net GND: Q601.3 (E), RV201.3
Other:
- note added: "Amplitude Adjust"
- title: (none) -> Pulse Output Driver
