File: Lab_06/Kicad_Files/Lab06.kicad_sch (KiCad schematic)
At the start: 74 parts, among them J1 Banana Jack, J2 Banana Jack, J3 Banana Jack, J4 Banana Jack, J5 Banana Jack, J6 Banana Jack, Q201 PNP, Q202 NPN, Q203 NPN, Q204 NPN, Q601 NPN, SW201 RANGE, U201 LM324A, U4 LF356, U401 LM324A, U5 LF356, U501 LM393

Commit message: Complete Revision 3 Lab 6 Schematic
Parts:
- removed Q201 (x2): PNP, symbol Simulation_SPICE:PNP
- removed Q202 (x2): NPN, symbol Simulation_SPICE:NPN
- removed R203: 100R, symbol Device:R
- removed R206: 1K5, symbol Device:R
- removed R501: 2K2, symbol Device:R
- removed R602: 22R, symbol Device:R
- removed RV201: 100R, symbol Device:R_Potentiometer
- removed U4: LF356, symbol Amplifier_Operational:LF356
- added C10, C11, C12, C3, C9: 0.1uF, symbol Device:C
- added Q6, Q8: NPN, symbol Simulation_SPICE:NPN
- added Q7, Q9: PNP, symbol Simulation_SPICE:PNP
- added R12, R17: 100K, symbol Device:R
- added R13: 470R, symbol Device:R
- added R14: 15K, symbol Device:R
- added R16: 1K, symbol Device:R
- added R19: 680K, symbol Device:R
- added R28: 560K, symbol Device:R
- added R31: 47K, symbol Device:R
- added R34: 560R, symbol Device:R
- added RV3: 1K, symbol Device:R_Potentiometer_Trim
- added RV5: 100K, symbol Device:R_Potentiometer
- added U2: TL082, symbol Amplifier_Operational:TL082
- C4: renamed from C1; value 0.01uF -> 0.1uF
- C5: renamed from C2; value 0.01uF -> 0.1uF
- R2: renamed from R202; value 1K -> 100K
- R29: renamed from R501; value 2K2 -> 100R
- R3: renamed from R203; value 1K -> 100K
- R33: renamed from R4; value 6K8 -> 5K6
- R35, R36, R37: renamed from R201; value 1K -> 68K
- R4: renamed from R205; value 1K -> 100K
- RV6: renamed from RV201; value 1K -> 2K
- RV7: renamed from RV201; value 10K -> 100K
- renumbered C201 to C1, C202 to C2, C601 to C6, C3 to C7, C4 to C8, D201 to D1, D202 to D2, D203 to D3, D204 to D4, D301 to D5, D302 to D6, Q201 to Q1, Q202 to Q2, Q203 to Q3, Q204 to Q4, Q601 to Q5, R203 to R1, R208 to R10, R209 to R11, R210 to R15, R301 to R18, R211 to R20, R204 to R21, R212 to R22, R206 to R23, R213 to R24, R214 to R25, R211 to R26, R215 to R27, R601 to R30, R4 to R32, R206 to R5, R206 to R6, R207 to R7, R207 to R8, R207 to R9, RV201 to RV1, RV202 to RV2, RV201 to RV4, RV201 to RV8, SW201 to SW1, U201 to U1, U5 to U3, U501 to U4, U401 to U5
Connections:
- net +15V: now also RV1.1, RV2.3, RV4.1, RV7.3, C10.1, C11.1, C12.1, C3.1, C9.1, Q6.1 (C), Q8.1 (C), R31.1, U2.8 (V+); no longer RV2.1, RV7.1
- net -15V: now also RV2.1, RV7.1, C10.2, C12.2, C3.2, C9.2, Q9.1 (C), R14.2, U2.4 (V-); no longer RV2.3
- net GND: now also U1.3 (+), C11.2, Q7.1 (C), R13.1, RV5.3, U2.3 (+); no longer RV7.3, U1.12 (+)
- net PULSE_IN: now also Q6.3 (E), Q7.3 (E), R28.2; no longer RV4.1
- net SIN: now also U1.6 (-), U1.7, U1.9 (-), U5.9 (-), Q8.3 (E), Q9.3 (E), R12.1; no longer U1.1, U1.2 (-), U1.6 (-), U5.13 (-)
- net at Q5.1 (C): now also Q6.2 (B), Q7.2 (B), R34.2
- net at D1.1 (K), D2.2 (A), R22.2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: now also U1.8; no longer U1.7
- net at R2.2, R3.2, R4.1: now also U1.2 (-); no longer U1.13 (-)
- net at R4.2, R6.1: now also U1.1; no longer U1.14
- net at R20.1, R22.1: now also U1.10 (+); no longer U1.5 (+)
- net at D3.1 (K), D4.2 (A), SW1.2 (B): now also R16.1; no longer Q3.1 (C), U1.3 (+)
- net at RV6.1: now also R33.1; no longer R32.2
- net at RV6.3: now also R32.2; no longer R33.1
- net at R37.2, U5.7: now also U5.10 (+); no longer U5.12 (+)
- net at RV4.2, U4.3 (+): now also R28.1
- net at R3.1, RV1.2: now also U1.12 (+); no longer U1.10 (+)
- net at RV7.2: now also U5.12 (+); no longer U5.10 (+)
- net at U4.2 (-): now also R19.2, U2.1
- new net: R12.2, R17.1, R19.1, U2.2 (-)
- new net: Q8.2 (B), Q9.2 (B), U5.8
- new net: Q3.1 (C), R16.2, U1.5 (+)
- new net: R5.1, U1.13 (-), U1.14
- new net: R13.2, RV3.1
- new net: R17.2, RV3.2
- new net: R14.1, RV3.3
- new net: R31.2, RV5.1
- new net: RV5.2, U2.5 (+)
- new net: R34.1, U2.6 (-), U2.7
- new net: R36.1, U5.13 (-), U5.14
Other:
- note added: "0V to 15V"
- note added: "15V to -8V"
- note added: "Input Zero Trim"
- note added: "Place near U3"
- note added: "Power Input & IC Power"
- note added: "Pulse Generator"
- note removed: "-8V to 15V"
- note removed: "0V to 14V"
- note removed: "Power Supply & IC Power"
- note removed: "Pulse Width Modulator"
- moved on the sheet: C1, C2, C4, C5, C6, C7, C8, D1, D2, D3, D4, D5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
