File: Lab_06/Kicad_Files/Lab06.kicad_sch (KiCad schematic)
At the start: 85 parts, among them J1 Banana Jack, J2 Banana Jack, J3 Banana Jack, J4 Banana Jack, J5 Banana Jack, J6 Banana Jack, Q1 PNP, Q2 NPN, Q3 NPN, Q4 NPN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

Commit message: Submit Labs 6 & 7
Parts:
- removed C11: 0.1uF, symbol Device:C
- removed C6: 1000pF, symbol Device:C
- R29: value 100R -> 2K2
Changed lines of the file:
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@@
   (title_block
     (title "Basic Analog Function Generator")
-    (date "2024-02-29")
-    (rev "3")
+    (date "2024-03-07")
+    (rev "4")
     (company "ZAM Industries, LLC")
     (comment 1 "Drawn by: Mark Vaughn")
@@
   (junction (at 400.05 327.66) (diameter 0) (color 0 0 0 0)
   )
-  (junction (at 365.76 259.08) (diameter 0) (color 0 0 0 0)
-  )
   (junction (at 356.87 347.98) (diameter 0) (color 0 0 0 0)
   )
   (junction (at 215.9 109.22) (diameter 0) (color 0 0 0 0)
   )
-  (junction (at 438.15 335.28) (diameter 0) (color 0 0 0 0)
-  )
   (junction (at 201.93 223.52) (diameter 0) (color 0 0 0 0)
   )
@@
   (junction (at 378.46 97.79) (diameter 0) (color 0 0 0 0)
   )
-  (junction (at 438.15 320.04) (diameter 0) (color 0 0 0 0)
-  )
   (junction (at 191.77 106.68) (diameter 0) (color 0 0 0 0)
   )
@@
   (junction (at 53.34 127) (diameter 0) (color 0 0 0 0)
   )
-  (junction (at 350.52 259.08) (diameter 0) (color 0 0 0 0)
-  )
   (junction (at 53.34 87.63) (diameter 0) (color 0 0 0 0)
   )
@@
     (stroke (width 0) (type default))
   )
-  (wire (pts (xy 434.34 320.04) (xy 438.15 320.04))
-    (stroke (width 0) (type default))
-  )
   (wire (pts (xy 40.64 127) (xy 43.18 127))
     (stroke (width 0) (type default))
@@
     (stroke (width 0) (type default))
   )
-  (wire (pts (xy 434.34 335.28) (xy 438.15 335.28))
-    (stroke (width 0) (type default))
-  )
   (wire (pts (xy 191.77 95.25) (xy 300.99 95.25))
     (stroke (width 0) (type default))
   )
-  (wire (pts (xy 350.52 266.7) (xy 354.33 266.7))
-    (stroke (width 0) (type default))
-  )
   (wire (pts (xy 386.08 248.92) (xy 412.75 248.92))
     (stroke (width 0) (type default))
@@
     (stroke (width 0) (type default))
   )
-  (wire (pts (xy 365.76 259.08) (xy 378.46 259.08))
-    (stroke (width 0) (type default))
-  )
   (wire (pts (xy 175.26 109.22) (xy 173.99 109.22))
     (stroke (width 0) (type default))
@@
     (stroke (width 0) (type default))
   )
-  (wire (pts (xy 321.31 259.08) (xy 350.52 259.08))
+  (wire (pts (xy 321.31 259.08) (xy 354.33 259.08))
     (stroke (width 0) (type default))
   )
@@
     (stroke (width 0) (type default))
   )
-  (wire (pts (xy 350.52 259.08) (xy 354.33 259.08))
-    (stroke (width 0) (type default))
-  )
   (wire (pts (xy 491.49 204.47) (xy 491.49 207.01))
     (stroke (width 0) (type default))
@@
     (stroke (width 0) (type default))
   )
-  (wire (pts (xy 350.52 259.08) (xy 350.52 266.7))
-    (stroke (width 0) (type default))
-  )
   (wire (pts (xy 222.25 148.59) (xy 223.52 148.59))
     (stroke (width 0) (type default))
@@
     (stroke (width 0) (type default))
   )
-  (wire (pts (xy 365.76 259.08) (xy 365.76 266.7))
-    (stroke (width 0) (type default))
-  )
   (wire (pts (xy 469.9 125.73) (xy 469.9 127))
     (stroke (width 0) (type default))
@@
     (stroke (width 0) (type default))
   )
-  (wire (pts (xy 361.95 266.7) (xy 365.76 266.7))
-    (stroke (width 0) (type default))
-  )
   (polyline (pts (xy 41.275 124.46) (xy 40.64 125.73))
     (stroke (width 0) (type default))
@@
     (stroke (width 0) (type default))
   )
-  (wire (pts (xy 434.34 331.47) (xy 434.34 335.28))
-    (stroke (width 0) (type default))
-  )
   (wire (pts (xy 461.01 105.41) (xy 461.01 113.03))
     (stroke (width 0) (type default))
@@
     (stroke (width 0) (type default))
   )
-  (wire (pts (xy 434.34 320.04) (xy 434.34 323.85))
-    (stroke (width 0) (type default))
-  )
   (wire (pts (xy 93.98 207.01) (xy 96.52 209.55))
     (stroke (width 0) (type default))
@@
     (stroke (width 0) (type default))
   )
-  (wire (pts (xy 361.95 259.08) (xy 365.76 259.08))
+  (wire (pts (xy 361.95 259.08) (xy 378.46 259.08))
     (stroke (width 0) (type default))
   )
@@
       (effects (font (size 1.27 1.27)) (justify left))
     )
-    (property "Value" "100R" (at 248.92 276.86 0)
+    (property "Value" "2K2" (at 248.92 276.86 0)
       (effects (font (size 1.27 1.27)) (justify left))
     )
@@
     )
   )
-  (symbol (lib_id "Device:C") (at 358.14 266.7 90) (unit 1)
-    (in_bom yes) (on_board yes) (dnp no)
-    (property "Reference" "C6" (at 359.41 265.43 90)
-      (effects (font (size 1.27 1.27)) (justify right))
-    )
-    (property "Value" "1000pF" (at 359.41 267.97 90)
-      (effects (font (size 1.27 1.27)) (justify right))
-    )
-    (property "Footprint" "" (at 361.95 265.7348 0)
-      (effects (font (size 1.27 1.27)) hide)
-    )
-    (property "Datasheet" "~" (at 358.14 266.7 0)
-      (effects (font (size 1.27 1.27)) hide)
-    )
-    (pin "1")
-    (pin "2")
-    (instances
-      (project "Lab06"
-        (path "/37d0ecfa-1973-4a3c-8fc1-f7066c204731"
-          (reference "C6") (unit 1)
-        )
-      )
-    )
-  )
   (symbol (lib_id "power:GND") (at 59.69 134.62 0) (unit 1)
     (in_bom yes) (on_board yes) (dnp no)
@@
         )
       )
-    )
-  )
-  (symbol (lib_id "Device:C") (at 434.34 327.66 0) (mirror y) (unit 1)
-    (in_bom yes) (on_board yes) (dnp no)
-    (property "Reference" "C11" (at 433.705 325.12 0)
-      (effects (font (size 1.27 1.27)) (justify left))
-    )
-    (property "Value" "0.1uF" (at 433.705 330.2 0)
-      (effects (font (size 1.27 1.27)) (justify left))
-    )
-    (property "Footprint" "" (at 433.3748 331.47 0)
-      (effects (font (size 1.27 1.27)) hide)
-    )
-    (property "Datasheet" "~" (at 434.34 327.66 0)
-      (effects (font (size 1.27 1.27)) hide)
-    )
-    (pin "1")
-    (pin "2")
-    (instances
-      (project "Lab06"
-        (path "/37d0ecfa-1973-4a3c-8fc1-f7066c204731"
-          (reference "C11") (unit 1)
-        )
-      )
