File: Lab_08/KiCad Files/Lab_08.kicad_sch (KiCad schematic)
At the start: 0 parts

Commit message: Continue Lab 8
Other:
- added sheet Full Schematic (04_TXRXFullSchema.kicad_sch)
- added sheet Receiver Timing Diagram (02_RXTiming.kicad_sch)
- added sheet System Block Diagram (03_TXRXBlocks.kicad_sch)
- note added: "12.5V"
- note added: "12V"
- note added: "2.5V"
- note added: "CYAN: Comparator Output"
- note added: "GREEN: 100Hz - 1KHz Tri. Oscillator"
- note added: "ORANGE: Input Signal"
- note added: "PAGE 2: RX TIMING DIAGRAM"
- note added: "PAGE 3: TX/RX BLOCK DIAGRAM"
- note added: "PAGE 4: FULL SYSTEM SCHEMATIC"
- company: (none) -> ZAM Industries, LLC
- title: (none) -> PWM Modulator/Transmitter Timing Diagram

Commit message: Complete Lab 8 First Revision Schema
Other:
- note added: "GREEN: 1KHz - 10KHz Tri. Oscillator"
- note removed: "12V"
- note removed: "GREEN: 100Hz - 1KHz Tri. Oscillator"
Changed lines of the file:
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@@
     (stroke (width 0) (type dot) (color 128 77 0 1))
   )
-  (polyline (pts (xy 226.06 108.585) (xy 237.49 108.585))
+  (polyline (pts (xy 226.06 102.235) (xy 237.49 102.235))
     (stroke (width 0.3175) (type default) (color 0 194 194 1))
   )
@@
     (stroke (width 0.508) (type default) (color 221 133 0 1))
   )
-  (polyline (pts (xy 141.605 127.635) (xy 141.605 108.585))
+  (polyline (pts (xy 141.605 127.635) (xy 141.605 102.235))
     (stroke (width 0.3175) (type default) (color 0 194 194 1))
   )
-  (polyline (pts (xy 141.605 108.585) (xy 168.275 108.585))
+  (polyline (pts (xy 141.605 102.235) (xy 168.275 102.235))
     (stroke (width 0.3175) (type default) (color 0 194 194 1))
   )
@@
     (stroke (width 0) (type dot) (color 194 0 0 1))
   )
-  (polyline (pts (xy 168.275 108.585) (xy 168.275 127.635))
+  (polyline (pts (xy 168.275 102.235) (xy 168.275 127.635))
     (stroke (width 0.3175) (type default) (color 0 194 194 1))
   )
@@
     (stroke (width 0.3175) (type default) (color 0 194 194 1))
   )
-  (polyline (pts (xy 237.49 108.585) (xy 237.49 127.635))
+  (polyline (pts (xy 237.49 102.235) (xy 237.49 127.635))
     (stroke (width 0.3175) (type default) (color 0 194 194 1))
   )
@@
     (stroke (width 0.3175) (type solid) (color 0 194 0 1))
   )
-  (polyline (pts (xy 184.15 127.635) (xy 184.15 108.585))
+  (polyline (pts (xy 184.15 127.635) (xy 184.15 102.235))
     (stroke (width 0.3175) (type default) (color 0 194 194 1))
   )
@@
     (stroke (width 0.508) (type default) (color 221 133 0 1))
   )
-  (polyline (pts (xy 86.995 108.585) (xy 277.495 108.585))
-    (stroke (width 0) (type dot) (color 194 0 0 1))
-  )
   (polyline (pts (xy 99.06 62.865) (xy 118.11 76.835))
     (stroke (width 0.3175) (type solid) (color 0 194 0 1))
   )
-  (polyline (pts (xy 184.15 108.585) (xy 202.565 108.585))
+  (polyline (pts (xy 184.15 102.235) (xy 202.565 102.235))
     (stroke (width 0.3175) (type default) (color 0 194 194 1))
   )
@@
     (stroke (width 0.3175) (type solid) (color 0 194 0 1))
   )
-  (polyline (pts (xy 99.695 127.635) (xy 99.695 108.585))
+  (polyline (pts (xy 99.695 127.635) (xy 99.695 102.235))
     (stroke (width 0.3175) (type default) (color 0 194 194 1))
   )
-  (polyline (pts (xy 268.605 127.635) (xy 268.605 108.585))
+  (polyline (pts (xy 268.605 127.635) (xy 268.605 102.235))
     (stroke (width 0.3175) (type default) (color 0 194 194 1))
   )
@@
     (stroke (width 0) (type dot) (color 194 0 0 1))
   )
-  (polyline (pts (xy 202.565 108.585) (xy 202.565 127.635))
+  (polyline (pts (xy 202.565 102.235) (xy 202.565 127.635))
     (stroke (width 0.3175) (type default) (color 0 194 194 1))
   )
@@
     (stroke (width 0.3175) (type dash) (color 0 194 0 1))
   )
-  (polyline (pts (xy 99.695 108.585) (xy 133.35 108.585))
+  (polyline (pts (xy 99.695 102.235) (xy 133.35 102.235))
     (stroke (width 0.3175) (type default) (color 0 194 194 1))
   )
@@
     (stroke (width 0.3175) (type dash) (color 0 194 0 1))
   )
-  (polyline (pts (xy 226.06 127.635) (xy 226.06 108.585))
+  (polyline (pts (xy 226.06 127.635) (xy 226.06 102.235))
     (stroke (width 0.3175) (type default) (color 0 194 194 1))
   )
-  (polyline (pts (xy 133.35 108.585) (xy 133.35 127.635))
+  (polyline (pts (xy 133.35 102.235) (xy 133.35 127.635))
     (stroke (width 0.3175) (type default) (color 0 194 194 1))
   )
@@
     (stroke (width 0) (type dot) (color 194 0 0 1))
   )
-  (polyline (pts (xy 268.605 108.585) (xy 271.78 108.585))
+  (polyline (pts (xy 268.605 102.235) (xy 271.78 102.235))
     (stroke (width 0.3175) (type default) (color 0 194 194 1))
   )
@@
     (stroke (width 0.3175) (type dash) (color 0 194 0 1))
   )
-  (polyline (pts (xy 271.78 108.585) (xy 271.78 127.635))
+  (polyline (pts (xy 271.78 102.235) (xy 271.78 127.635))
     (stroke (width 0.3175) (type default) (color 0 194 194 1))
   )
@@
     (effects (font (size 1.27 1.27) italic (color 194 0 0 1)) (justify left bottom))
   )
-  (text "GREEN: 100Hz - 1KHz\nTri. Oscillator" (at 74.93 79.375 0)
+  (text "GREEN: 1KHz - 10KHz\nTri. Oscillator" (at 74.93 79.375 0)
     (effects (font (size 3.175 3.175) (thickness 0.635) bold (color 0 194 0 1)) (justify right bottom))
   )
@@
     (effects (font (size 3.175 3.175) (thickness 0.635) bold (color 0 194 194 1)) (justify right bottom))
   )
-  (text "12V" (at 86.995 111.125 0)
-    (effects (font (size 1.27 1.27) italic (color 194 0 0 1)) (justify left bottom))
-  )
   (text "+15V" (at 92.075 59.69 0)

Commit message: Continue Lab 8
Other:
- added sheet Parts2and3 (05_Parts2and3.kicad_sch)
- note added: "PAGE 5: DEBOUNCE & TACHOMETER"
Changed lines of the file:
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@@
     (stroke (width 0.3175) (type solid) (color 0 194 0 1))
   )
-  (text "PAGE 4:\n\nFULL SYSTEM\nSCHEMATIC" (at 128.27 187.96 0)
+  (text "PAGE 4:\n\nFULL SYSTEM\nSCHEMATIC" (at 128.27 157.48 0)
     (effects (font (size 3.175 3.175) (thickness 0.635) bold) (justify left bottom))
   )
@@
     (effects (font (size 3.175 3.175) (thickness 0.635) bold (color 0 194 0 1)) (justify right bottom))
   )
-  (text "PAGE 3:\n\nTX/RX BLOCK\nDIAGRAM" (at 77.47 187.96 0)
+  (text "PAGE 3:\n\nTX/RX BLOCK\nDIAGRAM" (at 77.47 157.48 0)
     (effects (font (size 3.175 3.175) (thickness 0.635) bold) (justify left bottom))
   )
@@
     (effects (font (size 1.27 1.27) italic (color 194 0 0 1)) (justify left bottom))
   )
-  (text "PAGE 2:\n\nRX TIMING\nDIAGRAM" (at 26.67 187.96 0)
+  (text "PAGE 2:\n\nRX TIMING\nDIAGRAM" (at 26.67 157.48 0)
     (effects (font (size 3.175 3.175) (thickness 0.635) bold) (justify left bottom))
   )
@@
     (effects (font (size 1.27 1.27) italic) (justify left bottom))
   )
+  (text "PAGE 5:\n\nDEBOUNCE &\nTACHOMETER" (at 78.74 187.96 0)
+    (effects (font (size 3.175 3.175) (thickness 0.635) bold) (justify left bottom))
+  )
   (text "+15V" (at 92.075 104.775 0)
     (effects (font (size 1.27 1.27) italic (color 194 0 0 1)) (justify right bottom))
@@
     (stroke (width 0.1524) (type solid))
     (fill (color 0 0 0 0.0000))
-    (property "Sheetname" "System Block Diagram" (at 76.2 164.3884 0)
+    (property "Sheetname" "Parts2and3" (at 76.2 164.3884 0)
       (effects (font (size 1.27 1.27)) (justify left bottom) hide)
     )
-    (property "Sheetfile" "03_TXRXBlocks.kicad_sch" (at 76.2 191.0846 0)
+    (property "Sheetfile" "05_Parts2and3.kicad_sch" (at 76.2 191.0846 0)
+      (effects (font (size 1.27 1.27)) (justify left top))
+    )
+    (instances
+      (project "Lab_08"
+        (path "/1013cde2-6a46-4832-9725-5ce4a6675ae4" (page "5"))
+      )
+    )
+  )
+  (sheet (at 76.2 134.62) (size 38.1 25.4) (fields_autoplaced)
+    (stroke (width 0.1524) (type solid))
+    (fill (color 0 0 0 0.0000))
+    (property "Sheetname" "System Block Diagram" (at 76.2 133.9084 0)
+      (effects (font (size 1.27 1.27)) (justify left bottom) hide)
+    )
+    (property "Sheetfile" "03_TXRXBlocks.kicad_sch" (at 76.2 160.6046 0)
       (effects (font (size 1.27 1.27)) (justify left top))
     )
@@
     )
   )
-  (sheet (at 127 165.1) (size 38.1 25.4) (fields_autoplaced)
+  (sheet (at 127 134.62) (size 38.1 25.4) (fields_autoplaced)
     (stroke (width 0.1524) (type solid))
     (fill (color 0 0 0 0.0000))
-    (property "Sheetname" "Full Schematic" (at 127 164.3884 0)
+    (property "Sheetname" "Full Schematic" (at 127 133.9084 0)
       (effects (font (size 1.27 1.27)) (justify left bottom) hide)
     )
-    (property "Sheetfile" "04_TXRXFullSchema.kicad_sch" (at 127 191.0846 0)
+    (property "Sheetfile" "04_TXRXFullSchema.kicad_sch" (at 127 160.6046 0)
       (effects (font (size 1.27 1.27)) (justify left top))
     )
@@
     )
   )
-  (sheet (at 25.4 165.1) (size 38.1 25.4) (fields_autoplaced)
+  (sheet (at 25.4 134.62) (size 38.1 25.4) (fields_autoplaced)
     (stroke (width 0.1524) (type solid))
     (fill (color 0 0 0 0.0000))
-    (property "Sheetname" "Receiver Timing Diagram" (at 25.4 164.3884 0)
+    (property "Sheetname" "Receiver Timing Diagram" (at 25.4 133.9084 0)
       (effects (font (size 1.27 1.27)) (justify left bottom) hide)
     )
-    (property "Sheetfile" "02_RXTiming.kicad_sch" (at 25.4 191.0846 0)
+    (property "Sheetfile" "02_RXTiming.kicad_sch" (at 25.4 160.6046 0)
       (effects (font (size 1.27 1.27)) (justify left top))
     )
