File: Lab_08/KiCad Files/05_Parts2and3.kicad_sch (KiCad schematic)
At the start: 0 parts

Commit message: Finish Lab 8
Parts:
- added C?: 0.01uF, symbol Device:C
- added R?: 100K, symbol Device:R
- added U?: SE555P, Package_DIP:DIP-8_W7.62mm, symbol Timer:SE555P
- added U?: 4081, symbol 4xxx:4081
Connections:
- new net: C?.1, R?.2, U?.6 (THR), U?.7 (DIS)
- new net +15V: R?.1, U?.4 (R), U?.8 (VCC)
- new net GND: C?.2, U?.1 (GND)
- no-connect marks 0 -> 1
