File: Lab_11/KiCad Files/Lab_11/Lab_11.kicad_sch (KiCad schematic)
At the start: 41 parts, among them M1 DC Motor, Q1 Q_NPN_EBC, Q2 IRF9Z24, U1 LM393, U2 TLV272, U3 NE555P, U4 TSDP341xx

Commit message: Complete Revision 1 of Lab 11
Parts:
- removed D2: 10V, symbol Device:D_Zener
- removed Q2: IRF9Z24, symbol Device:Q_PMOS_GDS
- removed R2: 5K6, Resistor_THT:R_Axial_DIN0207_L6.3mm_D2.5mm_P7.62mm_Horizontal, symbol Device:R
- removed R7: 18K, Resistor_THT:R_Axial_DIN0207_L6.3mm_D2.5mm_P7.62mm_Horizontal, symbol Device:R
- added Q2: IRF530, Package_TO_SOT_THT:TO-220-3_Vertical, symbol Transistor_FET:IRF540N
- added R6: 15K, Resistor_THT:R_Axial_DIN0207_L6.3mm_D2.5mm_P7.62mm_Horizontal, symbol Device:R
- R10: renamed from R11; value 1M -> 680K
- R12: renamed from R13; value 1M -> 100K
- R14: renamed from R15; value 2.2M -> 220K
- R16: renamed from R17; value 2.2M -> 220K
- R17: renamed from R18; value 1M -> 120K
- R3: renamed from R4; value 100K -> 120K
- R4: renamed from R5; value 82K -> 68K
- R5: renamed from R6; value 100K -> 120K
- R7: renamed from R8; value 4K7 -> 2K2
- R9: renamed from R10; value 120K -> 100K
- renumbered D4 to D2, R12 to R11, R14 to R13, R16 to R15, R19 to R18, R20 to R19, R3 to R2, R23 to R20, R9 to R8
Connections:
- net GND: now also Q2.3 (S); no longer D2.2 (A), M1.2 (-)
- net VDD: no longer D1.1 (K), R1.2
- net V_Supply: now also D2.1 (K), M1.1 (+)
- net at R3.2, R5.1, U1.3 (+): now also R6.1
- net at RV1.1: now also D1.1 (K), R1.2
- net at R4.1, R7.2, U1.1: now also R6.2
- net at R20.2: now also Q2.1 (G)
- new net: D2.2 (A), M1.2 (-), Q2.2 (D)
Other:
- moved on the sheet: C2, D1, D2, M1, R1, R10, R12, R15, R2, R20, RV1, U2A

Commit message: Continue Lab 11 Schematic
Parts:
- removed D3: LD271, LED_THT:LED_D5.0mm_IRGrey, symbol LED:LD271
- removed U4: TSDP341xx, OptoDevice:Vishay_MOLD-3Pin, symbol Interface_Optical:TSDP341xx
- added D3: IR204, LED_THT:LED_D3.0mm_IRBlack, symbol LED:IR204A
- added Q3: PT204, LED_THT:LED_D5.0mm_Clear, symbol Sensor_Optical:BP103B
- added R23: 220K, Resistor_THT:R_Axial_DIN0207_L6.3mm_D2.5mm_P7.62mm_Horizontal, symbol Device:R
- added R9: 680K, Resistor_THT:R_Axial_DIN0207_L6.3mm_D2.5mm_P7.62mm_Horizontal, symbol Device:R
- U3: value NE555P -> SE555P
- renumbered R9 to R10, R10 to R11, R11 to R12, R12 to R13, R13 to R14, R14 to R15, R15 to R16, R16 to R17, R17 to R18, R18 to R19, R19 to R20, R20 to R21, R21 to R22, R22 to R24
Connections:
- net GND: now also D3.1 (K), Q3.2 (E)
- net VDD: now also U3.4 (R), R23.1
- net at C6.2: now also Q3.1 (C), R23.2
- net at C2.1, R8.1, U2.1: now also R9.2
- net at R11.1, R13.2, U2.2 (-): now also R9.1
- net at R24.2: now also D3.2 (A)
Other:
- moved on the sheet: R24

Commit message: Lab 11 Revision 3 Update
Parts:
- removed R16: 1K, Resistor_THT:R_Axial_DIN0207_L6.3mm_D2.5mm_P7.62mm_Horizontal, symbol Device:R
- added Q2: Q_PNP_EBC, symbol Device:Q_PNP_EBC
- R22: renamed from R23; value 220K -> 10K
- RV1: footprint (none) -> SamacSys_Parts:3386P1503
- U1, U2: footprint (none) -> Package_DIP:DIP-8_W7.62mm
- renumbered Q2 to Q3, Q3 to Q4, R17 to R16, R18 to R17, R19 to R18, R20 to R19, R21 to R20, R22 to R21, R24 to R23
Connections:
- net GND: now also Q2.3 (C); no longer Q1.1 (E)
- net V_Supply: now also Q1.3 (C)
- net at R20.1: now also Q1.1 (E), Q2.1 (E); no longer Q1.3 (C)
- net at Q1.2 (B), R14.2: now also Q2.2 (B)
Other:
- moved on the sheet: C1, C2, C3, C4, C5, C6, D1, D2, D3, M1, Q1, Q3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

Commit message: Lab 11 Revision 4
Parts:
- removed U1: LM393, Package_DIP:DIP-8_W7.62mm, symbol Comparator:LM393
- added R22: 4K7, Resistor_THT:R_Axial_DIN0207_L6.3mm_D2.5mm_P7.62mm_Horizontal, symbol Device:R
- added R23: 33K, Resistor_THT:R_Axial_DIN0207_L6.3mm_D2.5mm_P7.62mm_Horizontal, symbol Device:R
- added R24: 47K, Resistor_THT:R_Axial_DIN0207_L6.3mm_D2.5mm_P7.62mm_Horizontal, symbol Device:R
- added R25: 27K, Resistor_THT:R_Axial_DIN0207_L6.3mm_D2.5mm_P7.62mm_Horizontal, symbol Device:R
- added U1: LM339, symbol Comparator:LM339
- R13: value 100K -> 10K
- R26: renamed from R22; value 10K -> 220K
- renumbered R23 to R27
Connections:
- net GND: now also R25.2, U1.12 (V-)
- net VDD: now also R22.1, R24.1, U1.3 (V+)
- net at U2.5 (+): now also C3.2, R15.1, R16.2; no longer R17.2
- net at Q4.1 (C), R26.2: now also U1.10 (-); no longer C6.2
- net at R3.2, R5.1, R6.1: now also U1.5 (+)
- net at R10.2, R12.2, R14.1: now also U1.1
- net at R10.1, R8.2: now also U1.7 (+)
- net at R4.1, R6.2, R7.2: now also U1.2
- net at C1.1, R4.2: now also U1.4 (-), U1.6 (-)
- new net: R17.2, U2.6 (-)
- new net: R23.1, R24.2, R25.1, U1.11 (+)
- new net: C6.2, R22.2, R23.2, U1.13
Other:
- moved on the sheet: D3, Q4, R26, R27, U2B

Commit message: Finalize lab 11, add labs 12 & 13
Parts:
- removed R15: 220K, Resistor_THT:R_Axial_DIN0207_L6.3mm_D2.5mm_P7.62mm_Horizontal, symbol Device:R
- removed R18, R19: 10K, Resistor_THT:R_Axial_DIN0207_L6.3mm_D2.5mm_P7.62mm_Horizontal, symbol Device:R
- added C4: 0.22uF, symbol Device:C
- renumbered C4 to C5, C5 to C6, C6 to C7, R16 to R15, R17 to R16, R20 to R17, R21 to R18, R22 to R19, R23 to R20, R24 to R21, R25 to R22, R26 to R23, R27 to R24
Connections:
- net GND: now also C4.2
- net at R16.1: now also C4.1
