File: Lab_12/KiCad Files/Lab_12.kicad_pcb (KiCad board)
At the start: 2 copper layers, 182.9 x 114.3 mm, 64 parts, among them M1 DC Motor, Q1 2N4401, SW1 CCW, SW2 CW, U1 TLV272, U2 TLV274, U3 CD40106, U4 LM339, U5 4053, U6 L293D

Commit message: Finish Lab 12 Breadboard Layout
Parts:
- C8: footprint Capacitor_THT:C_Disc_D9.0mm_W2.5mm_P5.00mm -> Capacitor_THT:C_Disc_D9.0mm_W5.0mm_P7.50mm
- D2: footprint Diode_THT:D_A-405_P7.62mm_Horizontal -> Diode_THT:D_A-405_P2.54mm_Vertical_AnodeUp
- R12, R25, R31, R32, R6: footprint Resistor_THT:R_Axial_DIN0207_L6.3mm_D2.5mm_P7.62mm_Horizontal -> Resistor_THT:R_Axial_DIN0207_L6.3mm_D2.5mm_P5.08mm_Vertical
- R13, R24, R28, R33, R34, R5: footprint Resistor_THT:R_Axial_DIN0207_L6.3mm_D2.5mm_P7.62mm_Horizontal -> Resistor_THT:R_Axial_DIN0207_L6.3mm_D2.5mm_P10.16mm_Horizontal
- R14, R17, R18, R21, R22: footprint Resistor_THT:R_Axial_DIN0207_L6.3mm_D2.5mm_P7.62mm_Horizontal -> Resistor_THT:R_Axial_DIN0207_L6.3mm_D2.5mm_P2.54mm_Vertical
- R19, R23: footprint Resistor_THT:R_Axial_DIN0207_L6.3mm_D2.5mm_P7.62mm_Horizontal -> Resistor_THT:R_Axial_DIN0207_L6.3mm_D2.5mm_P15.24mm_Horizontal
- moved SC1 345.8 mm to (91.4, 76.2), turned to -90 degrees
- moved C9 344.4 mm to (91.4, 78.7)
- moved R34 344.4 mm to (86.4, 81.3)
- moved R30 338.3 mm to (78.7, 55.9), turned to 180 degrees
- moved R33 335.3 mm to (83.8, 81.3)
- moved R32 333.6 mm to (78.7, 76.2)
- moved C8 331.8 mm to (78.7, 61.0), turned to 180 degrees
- moved D2 331.1 mm to (78.7, 73.7)
- moved R26 327.9 mm to (78.7, 58.4), turned to 0 degrees
- moved R27 310.9 mm to (96.5, 58.4)
- moved R22 308.6 mm to (86.4, 61.0)
- moved RV5 307.2 mm to (99.1, 63.5), turned to 0 degrees
- moved R23 297.6 mm to (106.7, 53.3), turned to 180 degrees
- moved C6 272.7 mm to (121.8, 55.9)
- moved R21 267.2 mm to (124.5, 61.0), turned to 180 degrees
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Connections:
- U3 pad 1: Net-(C7-Pad1) -> GND
- U3 pad 11: unconnected-(U3-Pad11) -> GND
- U3 pad 2: Net-(R29-Pad2) -> unconnected-(U3-Pad2)
- U3 pad 3: unconnected-(U3-Pad3) -> GND
- U3 pad 5: unconnected-(U3-Pad5) -> Net-(C7-Pad1)
- U3 pad 6: unconnected-(U3-Pad6) -> Net-(R29-Pad2)
Routing:
- net (no net): track 1506.2 -> 1323.3 mm
- net Net-(D2-K): track 10.2 -> 166.2 mm, vias 0 -> 6
- net Net-(R20-Pad1): track 10.2 -> 126.1 mm, vias 0 -> 6
- net Net-(U6-4A): track 30.5 -> 145.4 mm, vias 0 -> 10
- net Net-(U5-X): track 10.2 -> 107.0 mm, vias 0 -> 6
- net Net-(U5-X0): track 20.3 -> 96.1 mm, vias 0 -> 4
- net Net-(U6-3A): track 30.5 -> 100.1 mm, vias 0 -> 2
- net Net-(U2A--): track 10.2 -> 68.6 mm, vias 0 -> 4
- net +6V: track 788.6 -> 844.7 mm, vias 30 -> 34
- net GND: track 1137.5 -> 1179.7 mm, vias 46 -> 56
- net Net-(R17-Pad1): track 20.3 -> 61.0 mm, vias 0 -> 4
- net Net-(R19-Pad1): track 10.2 -> 44.2 mm, vias 0 -> 4
- net Net-(U2D--): track 10.2 -> 43.2 mm, vias 0 -> 4
- net Net-(U2B--): track 10.2 -> 43.2 mm, vias 0 -> 4
- net Net-(U5-X1): track 20.3 -> 51.3 mm, vias 0 -> 2
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
Commit message: Finish Lab 12
Parts:
- removed the R15 at (149.9, 116.8)
- added R14: 2K2, Resistor_THT:R_Axial_DIN0207_L6.3mm_D2.5mm_P10.16mm_Horizontal, F.Cu at (193.0, 43.2)
- added R20: 120K, Resistor_THT:R_Axial_DIN0207_L6.3mm_D2.5mm_P10.16mm_Horizontal, F.Cu at (198.1, 43.2)
- added R21: 120K, Resistor_THT:R_Axial_DIN0207_L6.3mm_D2.5mm_P10.16mm_Horizontal, F.Cu at (198.1, 55.9)
- C3: value 220pF -> 100pF
- R16: value 1M5 -> 15K; footprint Resistor_THT:R_Axial_DIN0207_L6.3mm_D2.5mm_P7.62mm_Horizontal -> Resistor_THT:R_Axial_DIN0207_L6.3mm_D2.5mm_P5.08mm_Vertical
- R27: renamed from R25; footprint Resistor_THT:R_Axial_DIN0207_L6.3mm_D2.5mm_P5.08mm_Vertical -> Resistor_THT:R_Axial_DIN0207_L6.3mm_D2.5mm_P15.24mm_Horizontal
- moved R16 68.4 mm to (198.1, 58.4), turned to 180 degrees
- moved RV1 56.4 mm to (165.1, 58.4), turned to -90 degrees
- moved RV6 5.68 mm to (208.3, 58.4)
- moved R27 5.08 mm to (203.2, 61.0)
- renumbered R14 to R15, R20 to R22, R21 to R23, R22 to R24, R23 to R25, R24 to R26, R26 to R28, R27 to R29, R28 to R30, R29 to R31, R30 to R32, R31 to R33, R32 to R34, R33 to R35, R34 to R36
Connections:
- R16 pad 1: Net-(R16-Pad1) -> Net-(U4C-+)
- R16 pad 2: GND -> Net-(U5-X1)
- R27 pad 1: Net-(U4C-+) -> Net-(U4D-+)
- R30 pad 2: Net-(R28-Pad2) -> Net-(R30-Pad2)
- RV1 pad 1: Net-(R15-Pad2) -> +6V
- RV1 pad 2: Net-(RV1-Pad2) -> Net-(U4C--)
- RV1 pad 3: Net-(R16-Pad1) -> GND
- RV6 pad 1: Net-(R28-Pad2) -> GND
- RV6 pad 2: Net-(U4C-+) -> Net-(U4D-+)
- RV6 pad 3: GND -> Net-(R30-Pad2)
- U3 pad 12: Net-(U5-X1) -> unconnected-(U3-Pad12)
- U3 pad 13: Net-(RV1-Pad2) -> GND
- U4 pad 10: Net-(D2-K) -> Net-(U4C--)
- U4 pad 13: Net-(U5-A) -> Net-(U5-X1)
- U4 pad 14: unconnected-(U4-Pad14) -> Net-(U5-A)
- U4 pad 8: unconnected-(U4D---Pad8) -> Net-(D2-K)
- U4 pad 9: unconnected-(U4D-+-Pad9) -> Net-(U4D-+)
Routing:
- net Net-(RV1-Pad2): track 85.2 -> 0.00 mm, vias 2 -> 0
- net Net-(U4C--): track 0.00 -> 62.2 mm, vias 0 -> 5
- net Net-(R28-Pad2): track 29.4 -> 0.00 mm, vias 2 -> 0
- net Net-(U4D-+): track 0.00 -> 29.1 mm, vias 0 -> 2
- net Net-(U5-X1): track 51.3 -> 79.8 mm, vias 2 -> 4
- net +6V: track 844.7 -> 865.0 mm, vias 34 -> 36
- net GND: track 1179.7 -> 1197.5 mm, vias 56 -> 57
- net Net-(U4C-+): track 27.9 -> 10.2 mm, vias 2 -> 0
- net (no net): track 1323.3 -> 1313.2 mm
- net unconnected-(U4-Pad14): track 10.2 -> 0.00 mm
- net Net-(R30-Pad2): track 0.00 -> 10.2 mm
- net Net-(R16-Pad1): track 10.2 -> 0.00 mm
- net Net-(R15-Pad2): track 10.2 -> 0.00 mm
- net Net-(U6-4A): track 145.4 -> 138.4 mm, vias 10 -> 8
- net Net-(D2-K): track 166.2 -> 171.3 mm
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